Commit message: added turtlebot STL file for RViz

File: turtlebot3_description/urdf/turtlebot3_rplidar.urdf.xacro (robot description, xacro)
@@ -1,10 +1,4 @@
 <?xml version="1.0" ?>
 <robot name="turtlebot3" xmlns:xacro="http://ros.org/wiki/xacro">
-  <xacro:property name="astra_cam_px" value="0.13"/>
-  <xacro:property name="astra_cam_py" value="0.008"/>
-  <xacro:property name="astra_cam_pz" value="0.06"/>
-  <xacro:property name="astra_depth_rel_rgb_py" value="0.0250" />
-  <xacro:property name="astra_cam_rel_rgb_py"   value="-0.0125" />
-  <xacro:property name="astra_dae_display_scale"   value="0.5" />
   <xacro:property name="M_PI" value="3.1415926535897931" />
   <material name="black">
@@ -16,5 +10,5 @@
   <link name="base_footprint"/>
   <joint name="base_joint" type="fixed">
-    <origin xyz="0 0 0.033" rpy="0 0 0"/>
+    <origin xyz="0 0 0" rpy="0 0 0"/>
     <parent link="base_footprint"/>
     <child link="base_link" />
@@ -22,17 +16,18 @@
   <link name="base_link">
     <visual>
-      <origin xyz="0.06 0 0.007" rpy="0 0 0"/>
+      <origin xyz="0 0 0" rpy="0 0 0"/>
+      <geometry>
+        <mesh filename="package://turtlebot3_description/meshes/turtlebot3.stl" scale="0.001 0.001 0.001"/>
+      </geometry>
+      <material name="orange"/>
+    </visual>
+    <collision>
+      <origin xyz="0 0 0" rpy="0 0 0"/>
       <geometry>
         <box size="0.18 0.12 0.04"/>
       </geometry>
-    </visual>
-    <collision>
-      <origin xyz="0.06 0 0.007" rpy="0 0 0"/>
-      <geometry>
-        <box size="0.18 0.12 0.08"/>
-      </geometry>
     </collision>
     <inertial>
-      <origin xyz="0.06 0 0.007" rpy="0 0 0"/>
+      <origin xyz="0 0 0" rpy="0 0 0"/>
       <mass value="1"/>
       <inertia ixx="0.01" ixy="0.0" ixz="0.0"
@@ -44,5 +39,5 @@
     <parent link="base_link"/>
     <child link="wheel_left_link"/>
-    <origin xyz="0 0.08 0" rpy="-1.570796327 0 0"/>
+    <origin xyz="0.032 0.08 0.033" rpy="-1.570796327 0 0"/>
     <axis xyz="0 0 1"/>
   </joint>
@@ -53,5 +48,4 @@
         <cylinder length="0.018" radius="0.033"/>
       </geometry>
-      <material name="black"/>
     </visual>
     <collision>
@@ -72,5 +66,5 @@
     <parent link="base_link"/>
     <child link="wheel_right_link"/>
-    <origin xyz="0 -0.08 0" rpy="-1.570796327 0 0"/>
+    <origin xyz="0.032 -0.08 0.033" rpy="-1.570796327 0 0"/>
     <axis xyz="0 0 1"/>
   </joint>
@@ -81,5 +75,4 @@
         <cylinder length="0.018" radius="0.033"/>
       </geometry>
-      <material name="black"/>
     </visual>
     <collision>
@@ -98,5 +91,5 @@
   </link>
   <joint name="scan_joint" type="fixed">
-    <origin xyz="0 0 0.097" rpy="0 0 0"/>
+    <origin xyz="0 0 0.13025" rpy="0 0 0"/>
     <axis xyz="0 0 0"/>
     <parent link="base_link"/>
@@ -105,14 +98,13 @@
   <link name="base_scan">
     <visual>
-      <origin xyz="0 0 -0.02" rpy="0 0 0"/>
-      <geometry>
-        <cylinder length="0.06" radius="0.035"/>
+      <origin xyz="0 0 0.0204" rpy="0 0 0"/>
+      <geometry>125.86
+        <cylinder length="0.0408" radius="0.03785"/>
       </geometry>
-      <material name="black"/>
     </visual>
     <collision>
-      <origin rpy="0 0 -0.02" xyz="0 0 0"/>
+      <origin rpy="0 0 0" xyz="0 0 0"/>
       <geometry>
-        <cylinder length="0.06" radius="0.035"/>
+        <cylinder length="0.0408" radius="0.03785"/>
       </geometry>
     </collision>

Commit message: modified turtlebot3 model files

File: turtlebot3_description/urdf/turtlebot3_rplidar.urdf.xacro (robot description, xacro)
@@ -91,5 +91,5 @@
   </link>
   <joint name="scan_joint" type="fixed">
-    <origin xyz="0 0 0.13025" rpy="0 0 0"/>
+    <origin xyz="0 0 0.13925" rpy="0 0 0"/>
     <axis xyz="0 0 0"/>
     <parent link="base_link"/>
@@ -99,5 +99,5 @@
     <visual>
       <origin xyz="0 0 0.0204" rpy="0 0 0"/>
-      <geometry>125.86
+      <geometry>
         <cylinder length="0.0408" radius="0.03785"/>
       </geometry>
