Commit message: add sensor info for Intel RealSense R200

File: turtlebot3_description/urdf/turtlebot3_r200.urdf.xacro (robot description, xacro)
@@ -1,10 +1,11 @@
 <?xml version="1.0" ?>
 <robot name="turtlebot3" xmlns:xacro="http://ros.org/wiki/xacro">
-  <xacro:property name="astra_cam_px" value="0.13"/>
-  <xacro:property name="astra_cam_py" value="0.008"/>
-  <xacro:property name="astra_cam_pz" value="0.06"/>
-  <xacro:property name="astra_depth_rel_rgb_py" value="0.0250" />
-  <xacro:property name="astra_cam_rel_rgb_py" value="-0.0125" />
-  <xacro:property name="astra_dae_display_scale" value="0.5" />
+  <xacro:property name="r200_cam_offset_px" value="0.1" />
+  <xacro:property name="r200_cam_offset_py" value="-0.028" />
+  <xacro:property name="r200_cam_offset_pz" value="0.110" />
+  <xacro:property name="r200_cam_rgb_px" value="0.005"/>
+  <xacro:property name="r200_cam_rgb_py" value="0.018"/>
+  <xacro:property name="r200_cam_rgb_pz" value="0.013"/>
+  <xacro:property name="r200_cam_depth_offset" value="0.01"/>
   <xacro:property name="M_PI" value="3.1415926535897931" />
   <material name="black">
@@ -16,5 +17,5 @@
   <link name="base_footprint"/>
   <joint name="base_joint" type="fixed">
-    <origin xyz="0 0 0.033" rpy="0 0 0"/>
+    <origin xyz="0 0 0" rpy="0 0 0"/>
     <parent link="base_footprint"/>
     <child link="base_link" />
@@ -22,17 +23,18 @@
   <link name="base_link">
     <visual>
-      <origin xyz="0.06 0 0.007" rpy="0 0 0"/>
+      <origin xyz="0 0 0.061" rpy="0 0 0"/>
+      <geometry>
+        <box size="0.266 0.266 0.1"/>
+      </geometry>
+      <material name="orange"/>
+    </visual>
+    <collision>
+      <origin xyz="0 0 0" rpy="0 0 0"/>
       <geometry>
         <box size="0.18 0.12 0.04"/>
       </geometry>
-    </visual>
-    <collision>
-      <origin xyz="0.06 0 0.007" rpy="0 0 0"/>
-      <geometry>
-        <box size="0.18 0.12 0.08"/>
-      </geometry>
     </collision>
     <inertial>
-      <origin xyz="0.06 0 0.007" rpy="0 0 0"/>
+      <origin xyz="0 0 0" rpy="0 0 0"/>
       <mass value="1"/>
       <inertia ixx="0.01" ixy="0.0" ixz="0.0"
@@ -44,5 +46,5 @@
     <parent link="base_link"/>
     <child link="wheel_left_link"/>
-    <origin xyz="0 0.08 0" rpy="-1.570796327 0 0"/>
+    <origin xyz="0.065 0.140 0.033" rpy="-1.570796327 0 0"/>
     <axis xyz="0 0 1"/>
   </joint>
@@ -53,5 +55,4 @@
         <cylinder length="0.018" radius="0.033"/>
       </geometry>
-      <material name="black"/>
     </visual>
     <collision>
@@ -72,5 +73,5 @@
     <parent link="base_link"/>
     <child link="wheel_right_link"/>
-    <origin xyz="0 -0.08 0" rpy="-1.570796327 0 0"/>
+    <origin xyz="0.065 -0.140 0.033" rpy="-1.570796327 0 0"/>
     <axis xyz="0 0 1"/>
   </joint>
@@ -81,5 +82,4 @@
         <cylinder length="0.018" radius="0.033"/>
       </geometry>
-      <material name="black"/>
     </visual>
     <collision>
@@ -97,8 +97,36 @@
     </inertial>
   </link>
+  <!-- camera body -->
+  <joint name="camera_joint" type="fixed">
+    <origin xyz="${r200_cam_offset_px} ${r200_cam_offset_py} ${r200_cam_offset_pz}" rpy="0 0 0"/>
+    <parent link="base_link"/>
+    <child link="camera" />
+  </joint>
+  <link name="camera">
+    <visual>
+     <origin xyz="0 0 0" rpy="${M_PI/2} 0 ${M_PI/2}"/>
+      <geometry>
+       <mesh filename="package://turtlebot3_description/meshes/sensors/r200.dae" />
+      </geometry>
+    </visual>
+    <collision>
+      <origin xyz="0.0 0.0 0.0" rpy="0 0 0"/>
+      <geometry>
+        <box size="0.130 0.567 0.118"/>
+      </geometry>
+    </collision>-->
+    <!-- This inertial field needs doesn't contain reliable data!! -->
+   <inertial>
+      <mass value="0.564" />
+      <origin xyz="0 0 0" />
+      <inertia ixx="0.003881243" ixy="0.0" ixz="0.0"
+               iyy="0.000498940" iyz="0.0"
+               izz="0.003879257" />
+    </inertial>
+  </link>
+  <!-- RGB joints & links -->
   <joint name="camera_rgb_joint" type="fixed">
-    <origin xyz="${astra_cam_px} ${astra_cam_py} ${astra_cam_pz}"
-            rpy="0 0 0"/>
-    <parent link="base_link"/>
+    <origin xyz="${r200_cam_rgb_px} ${r200_cam_rgb_py} ${r200_cam_rgb_pz}" rpy="0 0 0"/>
+    <parent link="camera"/>
     <child link="camera_rgb_frame" />
   </joint>
@@ -110,41 +138,15 @@
   </joint>
   <link name="camera_rgb_optical_frame"/>
-  <joint name="camera_joint" type="fixed">
-    <origin xyz="0 ${astra_cam_rel_rgb_py} 0"
-            rpy="0 0 0"/>
-    <parent link="camera_rgb_frame"/>
-    <child link="camera_link"/>
-  </joint>
-  <link name="camera_link">
-    <visual>
-      <origin xyz="0 0 0" rpy="${M_PI/2} 0 ${M_PI/2}"/>
-      <geometry>
-        <mesh filename="package://turtlebot3_description/meshes/sensors/astra.dae" scale="${astra_dae_display_scale} ${astra_dae_display_scale} ${astra_dae_display_scale}"/>
-      </geometry>
-    </visual>
-    <collision>
-      <origin xyz="0.0 0.0 0.0" rpy="0 0 0" />
-      <geometry>
-      <box size="0.0400 0.1650 0.0300"/>
-    </geometry>
-    </collision>
-    <inertial>
-      <mass value="0.564" />
-      <origin xyz="0 0 0" />
-      <inertia ixx="0.003881243" ixy="0.0" ixz="0.0"
-               iyy="0.000498940" iyz="0.0"
-               izz="0.003879257" />
-    </inertial>
-  </link>
+  <!--Depth joints & links -->
   <joint name="camera_depth_joint" type="fixed">
-    <origin xyz="0 ${astra_depth_rel_rgb_py} 0" rpy="0 0 0" />
-    <parent link="camera_rgb_frame" />
-    <child link="camera_depth_frame" />
+      <origin xyz="0 ${r200_cam_depth_offset} 0" rpy="0 0 0" />
+      <parent link="camera_rgb_frame" />
+      <child link="camera_depth_frame" />
   </joint>
   <link name="camera_depth_frame"/>
   <joint name="camera_depth_optical_joint" type="fixed">
-    <origin xyz="0 0 0" rpy="${-M_PI/2} 0 ${-M_PI/2}" />
-    <parent link="camera_depth_frame" />
-    <child link="camera_depth_optical_frame" />
+      <origin xyz="0 0 0" rpy="${-M_PI/2} 0 ${-M_PI/2}" />
+      <parent link="camera_depth_frame" />
+      <child link="camera_depth_optical_frame" />
   </joint>
   <link name="camera_depth_optical_frame"/>

Commit message: modified the camera_link info

File: turtlebot3_description/urdf/turtlebot3_r200.urdf.xacro (robot description, xacro)
@@ -101,7 +101,7 @@
     <origin xyz="${r200_cam_offset_px} ${r200_cam_offset_py} ${r200_cam_offset_pz}" rpy="0 0 0"/>
     <parent link="base_link"/>
-    <child link="camera" />
+    <child link="camera_link" />
   </joint>
-  <link name="camera">
+  <link name="camera_link">
     <visual>
      <origin xyz="0 0 0" rpy="${M_PI/2} 0 ${M_PI/2}"/>
@@ -128,5 +128,5 @@
   <joint name="camera_rgb_joint" type="fixed">
     <origin xyz="${r200_cam_rgb_px} ${r200_cam_rgb_py} ${r200_cam_rgb_pz}" rpy="0 0 0"/>
-    <parent link="camera"/>
+    <parent link="camera_link"/>
     <child link="camera_rgb_frame" />
   </joint>
