Commit message: added new model of turtlebot3

File: turtlebot3_description/urdf/turtlebot3_lds.urdf.xacro (robot description, xacro)
@@ -18,5 +18,5 @@
       <origin xyz="0 0 0" rpy="0 0 0"/>
       <geometry>
-        <mesh filename="package://turtlebot3_description/meshes/turtlebot3.stl" scale="0.001 0.001 0.001"/>
+        <mesh filename="package://turtlebot3_description/meshes/turtlebot3_basic.stl" scale="0.001 0.001 0.001"/>
       </geometry>
       <material name="orange"/>

File: turtlebot3_description/urdf/turtlebot3_r200.urdf.xacro (robot description, xacro)
@@ -23,15 +23,16 @@
   <link name="base_link">
     <visual>
-      <origin xyz="0 0 0.061" rpy="0 0 0"/>
+      <origin xyz="0 0 0.0" rpy="0 0 0"/>
+      <geometry>
+        <mesh filename="package://turtlebot3_description/meshes/turtlebot3_premium.stl" scale="0.001 0.001 0.001"/>
+      </geometry>
+      <material name="orange"/>
+    </visual>
+    <collision>
+      <origin xyz="0 0 0.0" rpy="0 0 0"/>
       <geometry>
         <box size="0.266 0.266 0.1"/>
       </geometry>
       <material name="orange"/>
-    </visual>
-    <collision>
-      <origin xyz="0 0 0" rpy="0 0 0"/>
-      <geometry>
-        <box size="0.18 0.12 0.04"/>
-      </geometry>
     </collision>
     <inertial>
