Commit message: modified basic and premium urdf

File: turtlebot3_description/urdf/turtlebot3_basic.urdf.xacro (robot description, xacro)
@@ -2,23 +2,25 @@
 <robot name="turtlebot3" xmlns:xacro="http://ros.org/wiki/xacro">
   <xacro:property name="M_PI" value="3.1415926535897931" />
+  <!-- Init colour -->
   <material name="black">
     <color rgba="0.0 0.0 0.0 1.0"/>
   </material>
-  <material name="orange">
-    <color rgba="1.0 0.4 0.0 1.0"/>
+  <material name="light_black">
+    <color rgba="0.26 0.28 0.30 1.0"/>
   </material>
+  <!-- TurtleBot3 Base-->
   <link name="base_footprint"/>
   <joint name="base_joint" type="fixed">
-    <origin xyz="0 0 0" rpy="0 0 0"/>
     <parent link="base_footprint"/>
-    <child link="base_link" />
+    <child link="base_link"/>
+    <origin xyz="0 0 0.010" rpy="0 0 0"/>
   </joint>
   <link name="base_link">
     <visual>
-      <origin xyz="0 0 0" rpy="0 0 0"/>
+      <origin xyz="0 0 0.0" rpy="0 0 0"/>
       <geometry>
-        <mesh filename="package://turtlebot3_description/meshes/turtlebot3_basic.stl" scale="0.001 0.001 0.001"/>
+        <mesh filename="package://turtlebot3_description/meshes/pr30_tb3_basic.stl" scale="0.001 0.001 0.001"/>
       </geometry>
-      <material name="orange"/>
+      <material name="light_black"/>
     </visual>
     <collision>
@@ -36,16 +38,18 @@
     </inertial>
   </link>
+  <!-- TurtleBot3 Wheels-->
   <joint name="wheel_left_joint" type="continuous">
     <parent link="base_link"/>
     <child link="wheel_left_link"/>
-    <origin xyz="0.032 0.08 0.033" rpy="-1.570796327 0 0"/>
+    <origin xyz="0.032 0.08 0.023" rpy="${-M_PI*0.5} 0 0"/>
     <axis xyz="0 0 1"/>
   </joint>
   <link name="wheel_left_link">
     <visual>
-      <origin xyz="0 0 0" rpy="0 0 0"/>
+      <origin xyz="0 0 0" rpy="${M_PI*0.5} 0 0"/>
       <geometry>
-        <cylinder length="0.018" radius="0.033"/>
+        <mesh filename="package://turtlebot3_description/meshes/pr30_isw_tire_l.stl" scale="0.001 0.001 0.001"/>
       </geometry>
+      <material name="light_black"/>
     </visual>
     <collision>
@@ -66,13 +70,14 @@
     <parent link="base_link"/>
     <child link="wheel_right_link"/>
-    <origin xyz="0.032 -0.08 0.033" rpy="-1.570796327 0 0"/>
+    <origin xyz="0.032 -0.08 0.023" rpy="${-M_PI*0.5} 0 0"/>
     <axis xyz="0 0 1"/>
   </joint>
   <link name="wheel_right_link">
     <visual>
-      <origin xyz="0 0 0" rpy="0 0 0"/>
+      <origin xyz="0 0 0" rpy="${M_PI*0.5} 0 0"/>
       <geometry>
-        <cylinder length="0.018" radius="0.033"/>
+        <mesh filename="package://turtlebot3_description/meshes/pr30_isw_tire_r.stl" scale="0.001 0.001 0.001"/>
       </geometry>
+      <material name="light_black"/>
     </visual>
     <collision>
@@ -90,16 +95,51 @@
     </inertial>
   </link>
+  <joint name="caster_back_joint" type="fixed">
+    <parent link="base_link"/>
+    <child link="caster_back_link"/>
+    <origin xyz="-0.049 0 -0.004" rpy="${-M_PI*0.5} 0 0"/>
+  </joint>
+  <link name="caster_back_link">
+    <collision>
+      <origin rpy="0 0 0" xyz="0 0 0"/>
+      <geometry>
+        <box size="0.030 0.018 0.010"/>
+      </geometry>
+    </collision>
+    <inertial>
+      <origin xyz="0 0 0" />
+      <mass value="0.01" />
+      <inertia ixx="0.001" ixy="0.0" ixz="0.0"
+               iyy="0.001" iyz="0.0"
+               izz="0.001" />
+    </inertial>
+  </link>
+  <!-- TurtleBot3 Sensors-->
+  <joint name="gyro_joint" type="fixed">
+    <parent link="base_link"/>
+    <child link="gyro_link"/>
+    <origin xyz="0 0 0.058" rpy="0 0 0"/>
+  </joint>
+  <link name="gyro_link">
+    <inertial>
+      <origin xyz="0 0 0" />
+      <mass value="0.01" />
+      <inertia ixx="0.001" ixy="0.0" ixz="0.0"
+               iyy="0.001" iyz="0.0"
+               izz="0.001" />
+    </inertial>
+  </link>
   <joint name="scan_joint" type="fixed">
-    <origin xyz="0 0 0.13925" rpy="0 0 0"/>
-    <axis xyz="0 0 0"/>
     <parent link="base_link"/>
     <child link="base_scan"/>
+    <origin xyz="0 0 0.171" rpy="0 0 0"/>
   </joint>
   <link name="base_scan">
     <visual>
-      <origin xyz="0 0 0.0204" rpy="0 0 0"/>
+      <origin xyz="0 0 0.0" rpy="0 0 0"/>
       <geometry>
-        <cylinder length="0.0408" radius="0.03785"/>
+        <mesh filename="package://turtlebot3_description/meshes/sensors/lds.stl" scale="0.001 0.001 0.001"/>
       </geometry>
+      <material name="light_black"/>
     </visual>
     <collision>

File: turtlebot3_description/urdf/turtlebot3_premium.urdf.xacro (robot description, xacro)
@@ -9,15 +9,17 @@
   <xacro:property name="r200_cam_depth_offset" value="0.01"/>
   <xacro:property name="M_PI" value="3.1415926535897931" />
+  <!-- Init colour -->
   <material name="black">
     <color rgba="0.0 0.0 0.0 1.0"/>
   </material>
-  <material name="orange">
-    <color rgba="1.0 0.4 0.0 1.0"/>
+  <material name="light_black">
+    <color rgba="0.26 0.28 0.30 1.0"/>
   </material>
+  <!-- TurtleBot3 Base-->
   <link name="base_footprint"/>
   <joint name="base_joint" type="fixed">
-    <origin xyz="0 0 0" rpy="0 0 0"/>
     <parent link="base_footprint"/>
     <child link="base_link" />
+    <origin xyz="0 0 0.010" rpy="0 0 0"/>
   </joint>
   <link name="base_link">
@@ -25,7 +27,7 @@
       <origin xyz="0 0 0.0" rpy="0 0 0"/>
       <geometry>
-        <mesh filename="package://turtlebot3_description/meshes/turtlebot3_premium.stl" scale="0.001 0.001 0.001"/>
-      </geometry>
-      <material name="orange"/>
+        <mesh filename="package://turtlebot3_description/meshes/pr30_tb3_premium.stl" scale="0.001 0.001 0.001"/>
+      </geometry>
+      <material name="light_black"/>
     </visual>
     <collision>
@@ -34,5 +36,5 @@
         <box size="0.266 0.266 0.1"/>
       </geometry>
-      <material name="orange"/>
+      <material name="light_black"/>
     </collision>
     <inertial>
@@ -44,16 +46,46 @@
     </inertial>
   </link>
+  <!-- TurtleBot3 Wheels-->
   <joint name="wheel_left_joint" type="continuous">
     <parent link="base_link"/>
     <child link="wheel_left_link"/>
-    <origin xyz="0.065 0.140 0.033" rpy="-1.570796327 0 0"/>
+    <origin xyz="0.064 0.144 0.021" rpy="${-M_PI*0.5} 0 0"/>
     <axis xyz="0 0 1"/>
   </joint>
   <link name="wheel_left_link">
     <visual>
-      <origin xyz="0 0 0" rpy="0 0 0"/>
+      <origin xyz="0 0 0" rpy="${M_PI*0.5} 0 0"/>
+      <geometry>
+        <mesh filename="package://turtlebot3_description/meshes/pr30_isw_tire_l.stl" scale="0.001 0.001 0.001"/>
+      </geometry>
+      <material name="light_black"/>
+    </visual>
+    <collision>
+      <origin rpy="0 0 0" xyz="0 0 0"/>
       <geometry>
         <cylinder length="0.018" radius="0.033"/>
       </geometry>
+    </collision>
+    <inertial>
+      <origin xyz="0 0 0" />
+      <mass value="0.01" />
+      <inertia ixx="0.001" ixy="0.0" ixz="0.0"
+               iyy="0.001" iyz="0.0"
+               izz="0.001" />
+    </inertial>
+  </link>
+  <joint name="wheel_right_joint" type="continuous">
+    <parent link="base_link"/>
+    <child link="wheel_right_link"/>
+    <origin xyz="0.064 -0.144 0.021" rpy="${-M_PI*0.5} 0 0"/>
+    <axis xyz="0 0 1"/>
+  </joint>
+  <link name="wheel_right_link">
+    <visual>
+      <origin xyz="0 0 0" rpy="${M_PI*0.5} 0 0"/>
+      <geometry>
+        <mesh filename="package://turtlebot3_description/meshes/pr30_isw_tire_r.stl" scale="0.001 0.001 0.001"/>
+      </geometry>
+      <material name="light_black"/>
     </visual>
     <collision>
@@ -71,34 +103,88 @@
     </inertial>
   </link>
-  <joint name="wheel_right_joint" type="continuous">
-    <parent link="base_link"/>
-    <child link="wheel_right_link"/>
-    <origin xyz="0.065 -0.140 0.033" rpy="-1.570796327 0 0"/>
-    <axis xyz="0 0 1"/>
-  </joint>
-  <link name="wheel_right_link">
-    <visual>
-      <origin xyz="0 0 0" rpy="0 0 0"/>
-      <geometry>
-        <cylinder length="0.018" radius="0.033"/>
-      </geometry>
-    </visual>
-    <collision>
-      <origin rpy="0 0 0" xyz="0 0 0"/>
-      <geometry>
-        <cylinder length="0.018" radius="0.033"/>
-      </geometry>
-    </collision>
-    <inertial>
-      <origin xyz="0 0 0" />
-      <mass value="0.01" />
-      <inertia ixx="0.001" ixy="0.0" ixz="0.0"
-               iyy="0.001" iyz="0.0"
-               izz="0.001" />
-    </inertial>
-  </link>
-  <!-- camera body -->
+  <joint name="caster_back_right_joint" type="fixed">
+    <parent link="base_link"/>
+    <child link="caster_back_right_link"/>
+    <origin xyz="-0.113 -0.064 -0.004" rpy="${-M_PI*0.5} 0 0"/>
+  </joint>
+  <link name="caster_back_right_link">
+    <collision>
+      <origin rpy="0 0 0" xyz="0 0 0"/>
+      <geometry>
+        <box size="0.030 0.018 0.010"/>
+      </geometry>
+    </collision>
+    <inertial>
+      <origin xyz="0 0 0" />
+      <mass value="0.01" />
+      <inertia ixx="0.001" ixy="0.0" ixz="0.0"
+               iyy="0.001" iyz="0.0"
+               izz="0.001" />
+    </inertial>
+  </link>
+  <joint name="caster_back_left_joint" type="fixed">
+    <parent link="base_link"/>
+    <child link="caster_back_left_link"/>
+    <origin xyz="-0.113 0.064 -0.004" rpy="${-M_PI*0.5} 0 0"/>
+  </joint>
+  <link name="caster_back_left_link">
+    <collision>
+      <origin rpy="0 0 0" xyz="0 0 0"/>
+      <geometry>
+        <box size="0.030 0.018 0.010"/>
+      </geometry>
+    </collision>
+    <inertial>
+      <origin xyz="0 0 0" />
+      <mass value="0.01" />
+      <inertia ixx="0.001" ixy="0.0" ixz="0.0"
+               iyy="0.001" iyz="0.0"
+               izz="0.001" />
+    </inertial>
+  </link>
+  <!-- TurtleBot3 Sensors-->
+  <joint name="gyro_joint" type="fixed">
+    <parent link="base_link"/>
+    <child link="gyro_link"/>
+    <origin xyz="0.064 0 0.057" rpy="0 0 0"/>
+  </joint>
+  <link name="gyro_link">
+    <inertial>
+      <origin xyz="0 0 0" />
+      <mass value="0.01" />
+      <inertia ixx="0.001" ixy="0.0" ixz="0.0"
+               iyy="0.001" iyz="0.0"
+               izz="0.001" />
+    </inertial>
+  </link>
+  <joint name="scan_joint" type="fixed">
+    <parent link="base_link"/>
+    <child link="base_scan"/>
+    <origin xyz="0 0 0.121" rpy="0 0 0"/>
+  </joint>
+  <link name="base_scan">
+    <visual>
+      <origin xyz="0 0 0.0" rpy="0 0 0"/>
+      <geometry>
+        <mesh filename="package://turtlebot3_description/meshes/sensors/lds.stl" scale="0.001 0.001 0.001"/>
+      </geometry>
+      <material name="light_black"/>
+    </visual>
+    <collision>
+      <origin rpy="0 0 0" xyz="0 0 0"/>
+      <geometry>
+        <cylinder length="0.0408" radius="0.03785"/>
+      </geometry>
+    </collision>
+    <inertial>
+      <mass value="0.01" />
+      <origin xyz="0 0 0" />
+      <inertia ixx="0.001" ixy="0.0" ixz="0.0"
+               iyy="0.001" iyz="0.0"
+               izz="0.001" />
+    </inertial>
+  </link>
   <joint name="camera_joint" type="fixed">
-    <origin xyz="${r200_cam_offset_px} ${r200_cam_offset_py} ${r200_cam_offset_pz}" rpy="0 0 0"/>
+    <origin xyz="0.140 -0.065 0.084" rpy="0 0 0"/>
     <parent link="base_link"/>
     <child link="camera_link" />
@@ -106,5 +192,5 @@
   <link name="camera_link">
     <visual>
-     <origin xyz="0 0 0" rpy="${M_PI/2} 0 ${M_PI/2}"/>
+     <origin xyz="0 0 0" rpy="${M_PI*0.5} 0 ${M_PI*0.5}"/>
       <geometry>
        <mesh filename="package://turtlebot3_description/meshes/sensors/r200.dae" />

Commit message: modified file name

File: turtlebot3_description/urdf/turtlebot3_basic.urdf.xacro (robot description, xacro)
@@ -20,5 +20,5 @@
       <origin xyz="0 0 0.0" rpy="0 0 0"/>
       <geometry>
-        <mesh filename="package://turtlebot3_description/meshes/pr30_tb3_basic.stl" scale="0.001 0.001 0.001"/>
+        <mesh filename="package://turtlebot3_description/meshes/basic_base.stl" scale="0.001 0.001 0.001"/>
       </geometry>
       <material name="light_black"/>
@@ -49,5 +49,5 @@
       <origin xyz="0 0 0" rpy="${M_PI*0.5} 0 0"/>
       <geometry>
-        <mesh filename="package://turtlebot3_description/meshes/pr30_isw_tire_l.stl" scale="0.001 0.001 0.001"/>
+        <mesh filename="package://turtlebot3_description/meshes/left_tire.stl" scale="0.001 0.001 0.001"/>
       </geometry>
       <material name="light_black"/>
@@ -77,5 +77,5 @@
       <origin xyz="0 0 0" rpy="${M_PI*0.5} 0 0"/>
       <geometry>
-        <mesh filename="package://turtlebot3_description/meshes/pr30_isw_tire_r.stl" scale="0.001 0.001 0.001"/>
+        <mesh filename="package://turtlebot3_description/meshes/right_tire.stl" scale="0.001 0.001 0.001"/>
       </geometry>
       <material name="light_black"/>

File: turtlebot3_description/urdf/turtlebot3_premium.urdf.xacro (robot description, xacro)
@@ -27,5 +27,5 @@
       <origin xyz="0 0 0.0" rpy="0 0 0"/>
       <geometry>
-        <mesh filename="package://turtlebot3_description/meshes/pr30_tb3_premium.stl" scale="0.001 0.001 0.001"/>
+        <mesh filename="package://turtlebot3_description/meshes/premium_base.stl" scale="0.001 0.001 0.001"/>
       </geometry>
       <material name="light_black"/>
@@ -57,5 +57,5 @@
       <origin xyz="0 0 0" rpy="${M_PI*0.5} 0 0"/>
       <geometry>
-        <mesh filename="package://turtlebot3_description/meshes/pr30_isw_tire_l.stl" scale="0.001 0.001 0.001"/>
+        <mesh filename="package://turtlebot3_description/meshes/left_tire.stl" scale="0.001 0.001 0.001"/>
       </geometry>
       <material name="light_black"/>
@@ -85,5 +85,5 @@
       <origin xyz="0 0 0" rpy="${M_PI*0.5} 0 0"/>
       <geometry>
-        <mesh filename="package://turtlebot3_description/meshes/pr30_isw_tire_r.stl" scale="0.001 0.001 0.001"/>
+        <mesh filename="package://turtlebot3_description/meshes/right_tire.stl" scale="0.001 0.001 0.001"/>
       </geometry>
       <material name="light_black"/>

Commit message: update navigation

File: turtlebot3_description/urdf/turtlebot3_basic.urdf.xacro (robot description, xacro)
@@ -116,10 +116,10 @@
   </link>
   <!-- TurtleBot3 Sensors-->
-  <joint name="gyro_joint" type="fixed">
+<!--  <joint name="imu_joint" type="fixed">
     <parent link="base_link"/>
-    <child link="gyro_link"/>
-    <origin xyz="0 0 0.058" rpy="0 0 0"/>
+    <child link="imu_link"/>
+    <origin xyz="0.0 0 0.058" rpy="0 0 0"/>
   </joint>
-  <link name="gyro_link">
+  <link name="imu_link">
     <inertial>
       <origin xyz="0 0 0" />
@@ -129,5 +129,5 @@
                izz="0.001" />
     </inertial>
-  </link>
+  </link>-->
   <joint name="scan_joint" type="fixed">
     <parent link="base_link"/>
