Commit message: add lidar

File: turtlebot3_description/urdf/turtlebot3_waffle_pi_naked.urdf.xacro (robot description, xacro)
@@ -138,4 +138,32 @@
     <child link="camera_link"/>
   </joint>
+  <joint name="scan_joint" type="fixed">
+    <parent link="base_link"/>
+    <child link="base_scan"/>
+    <!-- <origin xyz="-0.064 0 0.121" rpy="0 0 0"/> -->
+    <origin xyz="-0.008 0 0.121" rpy="0 0 0"/>
+  </joint>
+  <link name="base_scan">
+    <visual>
+      <origin xyz="0 0 0.0" rpy="0 0 0"/>
+      <geometry>
+        <mesh filename="package://turtlebot3_description/meshes/sensors/lds.stl" scale="0.001 0.001 0.001"/>
+      </geometry>
+      <material name="dark"/>
+    </visual>
+    <collision>
+      <origin xyz="0.015 0 -0.003" rpy="0 0 0"/>
+      <geometry>
+        <cylinder length="0.0415" radius="0.055"/>
+      </geometry>
+    </collision>
+    <inertial>
+      <mass value="0.114" />
+      <origin xyz="0 0 0" />
+      <inertia ixx="0.001" ixy="0.0" ixz="0.0"
+               iyy="0.001" iyz="0.0"
+               izz="0.001" />
+    </inertial>
+  </link>
   <link name="camera_link">
     <collision>

Commit message: update scan param

File: turtlebot3_description/urdf/turtlebot3_waffle_pi_naked.urdf.xacro (robot description, xacro)
@@ -2,5 +2,5 @@
 <robot name="turtlebot3_waffle_pi" xmlns:xacro="http://ros.org/wiki/xacro">
   <xacro:include filename="$(find turtlebot3_description)/urdf/common_properties.xacro"/>
-  <xacro:include filename="$(find turtlebot3_description)/urdf/turtlebot3_waffle_pi_naked.gazebo.xacro"/>
+  <xacro:include filename="$(find turtlebot3_description)/urdf/turtlebot3_waffle_pi.gazebo.xacro"/>
   <link name="base_footprint"/>
   <joint name="base_joint" type="fixed">
@@ -141,6 +141,5 @@
     <parent link="base_link"/>
     <child link="base_scan"/>
-    <!-- <origin xyz="-0.064 0 0.121" rpy="0 0 0"/> -->
-    <origin xyz="-0.008 0 0.122" rpy="0 0 0"/>
+    <origin xyz="-0.025 0 0.122" rpy="0 0 0"/>
   </joint>
   <link name="base_scan">
@@ -155,5 +154,5 @@
       <origin xyz="0.015 0 -0.0065" rpy="0 0 0"/>
       <geometry>
-        <cylinder length="0.0315" radius="0.055"/>
+        <cylinder length="0.0315" radius="0.045"/>
       </geometry>
     </collision>
