Commit message: delete base_scan tag and add imu tag

File: turtlebot3_description/urdf/turtlebot3_waffle_naked.urdf.xacro (robot description, xacro)
@@ -131,46 +131,10 @@
     </inertial>
   </link>
-  <!-- TurtleBot3 Sensors-->
-<!--  <joint name="gyro_joint" type="fixed">
+  <joint name="imu_joint" type="fixed">
     <parent link="base_link"/>
-    <child link="gyro_link"/>
-    <origin xyz="0.064 0 0.057" rpy="0 0 0"/>
+    <child link="imu_link"/>
+    <origin xyz="0.0 0 0.068" rpy="0 0 0"/>
   </joint>
-  <link name="gyro_link">
-    <inertial>
-      <origin xyz="0 0 0" />
-      <mass value="0.01" />
-      <inertia ixx="0.001" ixy="0.0" ixz="0.0"
-               iyy="0.001" iyz="0.0"
-               izz="0.001" />
-    </inertial>
-  </link>-->
-<!--  <joint name="scan_joint" type="fixed">
-    <parent link="base_link"/>
-    <child link="base_scan"/>
-    <origin xyz="-0.064 0 0.121" rpy="0 0 0"/>
-  </joint>
-  <link name="base_scan">
-    <visual>
-      <origin xyz="0 0 0.0" rpy="0 0 0"/>
-      <geometry>
-        <mesh filename="package://turtlebot3_description/meshes/sensors/lds.stl" scale="0.001 0.001 0.001"/>
-      </geometry>
-      <material name="dark"/>
-    </visual>
-    <collision>
-      <origin rpy="0 0 0" xyz="0 0 0"/>
-      <geometry>
-        <cylinder length="0.0408" radius="0.070"/>
-      </geometry>
-    </collision>
-    <inertial>
-      <mass value="0.01" />
-      <origin xyz="0 0 0" />
-      <inertia ixx="0.001" ixy="0.0" ixz="0.0"
-               iyy="0.001" iyz="0.0"
-               izz="0.001" />
-    </inertial>
-  </link>-->
+  <link name="imu_link"/>
   <joint name="camera_joint" type="fixed">
     <origin xyz="0.064 -0.065 0.094" rpy="0 0 0"/>

Commit message: update scan param

File: turtlebot3_description/urdf/turtlebot3_waffle_naked.urdf.xacro (robot description, xacro)
@@ -137,4 +137,31 @@
   </joint>
   <link name="imu_link"/>
+  <joint name="scan_joint" type="fixed">
+    <parent link="base_link"/>
+    <child link="base_scan"/>
+    <origin xyz="-0.024 0 0.122" rpy="0 0 0"/>
+  </joint>
+  <link name="base_scan">
+    <visual>
+      <origin xyz="0 0 0.0" rpy="0 0 0"/>
+      <geometry>
+        <mesh filename="package://turtlebot3_description/meshes/sensors/lds.stl" scale="0.001 0.001 0.001"/>
+      </geometry>
+      <material name="dark"/>
+    </visual>
+    <collision>
+      <origin xyz="0.015 0 -0.0065" rpy="0 0 0"/>
+      <geometry>
+        <cylinder length="0.0315" radius="0.045"/>
+      </geometry>
+    </collision>
+    <inertial>
+      <mass value="0.114" />
+      <origin xyz="0 0 0" />
+      <inertia ixx="0.001" ixy="0.0" ixz="0.0"
+               iyy="0.001" iyz="0.0"
+               izz="0.001" />
+    </inertial>
+  </link>
   <joint name="camera_joint" type="fixed">
     <origin xyz="0.064 -0.065 0.094" rpy="0 0 0"/>

File: turtlebot3_description/urdf/turtlebot3_waffle_pi_naked.urdf.xacro (robot description, xacro)
@@ -133,13 +133,8 @@
   </joint>
   <link name="imu_link"/>
-  <joint name="camera_joint" type="fixed">
-    <origin xyz="0.073 -0.011 0.084" rpy="0 0 0"/>
-    <parent link="base_link"/>
-    <child link="camera_link"/>
-  </joint>
   <joint name="scan_joint" type="fixed">
     <parent link="base_link"/>
     <child link="base_scan"/>
-    <origin xyz="-0.025 0 0.122" rpy="0 0 0"/>
+    <origin xyz="-0.024 0 0.122" rpy="0 0 0"/>
   </joint>
   <link name="base_scan">
@@ -165,4 +160,9 @@
     </inertial>
   </link>
+  <joint name="camera_joint" type="fixed">
+    <origin xyz="0.073 -0.011 0.084" rpy="0 0 0"/>
+    <parent link="base_link"/>
+    <child link="camera_link"/>
+  </joint>
   <link name="camera_link">
     <collision>
