Commit message: update URDF

File: turtlebot3_description/urdf/turtlebot3_waffle.urdf.xacro (robot description, xacro)
@@ -29,5 +29,4 @@
         <box size="0.265 0.265 0.089"/>
       </geometry>
-      <material name="light_black"/>
     </collision>
     <inertial>

Commit message: update turtlebot3 waffle URDF

File: turtlebot3_description/urdf/turtlebot3_waffle.urdf.xacro (robot description, xacro)
@@ -177,5 +177,5 @@
   </link>
   <joint name="camera_joint" type="fixed">
-    <origin xyz="0.076 -0.065 0.084" rpy="0 0 0"/>
+    <origin xyz="0.064 -0.065 0.094" rpy="0 0 0"/>
     <parent link="base_link"/>
     <child link="camera_link"/>

Commit message: Fix the tf tree according to the one of realsense camera and commented out deprecated parameters.

File: turtlebot3_description/urdf/turtlebot3_waffle.urdf.xacro (robot description, xacro)
@@ -3,7 +3,9 @@
   <xacro:include filename="$(find turtlebot3_description)/urdf/common_properties.xacro"/>
   <xacro:include filename="$(find turtlebot3_description)/urdf/turtlebot3_waffle.gazebo.xacro"/>
-  <xacro:property name="r200_cam_offset_px" value="0.1" />
-  <xacro:property name="r200_cam_offset_py" value="-0.028" />
-  <xacro:property name="r200_cam_offset_pz" value="0.110" />
+  <!-- deprecated parameters -->
+  <!-- <xacro:property name="r200_cam_offset_px" value="0.1" /> -->
+  <!-- <xacro:property name="r200_cam_offset_py" value="-0.028" /> -->
+  <!-- <xacro:property name="r200_cam_offset_pz" value="0.110" /> -->
+  <!-- camera transformation parameters -->
   <xacro:property name="r200_cam_rgb_px" value="0.005"/>
   <xacro:property name="r200_cam_rgb_py" value="0.018"/>
@@ -207,6 +209,6 @@
   <link name="camera_rgb_optical_frame"/>
   <joint name="camera_depth_joint" type="fixed">
-      <origin xyz="0 ${r200_cam_depth_offset} 0" rpy="0 0 0"/>
-      <parent link="camera_rgb_frame"/>
+      <origin xyz="${r200_cam_rgb_px} ${r200_cam_rgb_py+r200_cam_depth_offset} ${r200_cam_rgb_pz}" rpy="0 0 0"/>
+      <parent link="camera_link"/>
       <child link="camera_depth_frame"/>
   </joint>

Commit message: edit collision

File: turtlebot3_description/urdf/turtlebot3_waffle.urdf.xacro (robot description, xacro)
@@ -98,5 +98,5 @@
   <link name="caster_back_right_link">
     <collision>
-      <origin rpy="0 0.001 0" xyz="0 0 0"/>
+      <origin xyz="0 0.001 0" rpy="0 0 0"/>
       <geometry>
         <box size="0.030 0.009 0.020"/>
@@ -118,5 +118,5 @@
   <link name="caster_back_left_link">
     <collision>
-      <origin rpy="0 0.001 0" xyz="0 0 0"/>
+      <origin xyz="0 0.001 0" rpy="0 0 0"/>
       <geometry>
         <box size="0.030 0.009 0.020"/>

File: turtlebot3_description/urdf/turtlebot3_waffle_naked.urdf.xacro (robot description, xacro)
@@ -98,5 +98,5 @@
   <link name="caster_back_right_link">
     <collision>
-      <origin rpy="0 0 0" xyz="0 0 0"/>
+      <origin xyz="0 0.001 0" rpy="0 0 0"/>
       <geometry>
         <box size="0.030 0.009 0.020"/>
@@ -118,5 +118,5 @@
   <link name="caster_back_left_link">
     <collision>
-      <origin rpy="0 0 0" xyz="0 0 0"/>
+      <origin xyz="0 0.001 0" rpy="0 0 0"/>
       <geometry>
         <box size="0.030 0.009 0.020"/>

File: turtlebot3_description/urdf/turtlebot3_waffle_pi.urdf.xacro (robot description, xacro)
@@ -94,5 +94,5 @@
   <link name="caster_back_right_link">
     <collision>
-      <origin rpy="0 0.001 0" xyz="0 0 0"/>
+      <origin xyz="0 0.001 0" rpy="0 0 0"/>
       <geometry>
         <box size="0.030 0.009 0.020"/>
@@ -114,5 +114,5 @@
   <link name="caster_back_left_link">
     <collision>
-      <origin rpy="0 0.001 0" xyz="0 0 0"/>
+      <origin xyz="0 0.001 0" rpy="0 0 0"/>
       <geometry>
         <box size="0.030 0.009 0.020"/>

File: turtlebot3_description/urdf/turtlebot3_waffle_pi_naked.urdf.xacro (robot description, xacro)
@@ -94,5 +94,5 @@
   <link name="caster_back_right_link">
     <collision>
-      <origin rpy="0 0.001 0" xyz="0 0 0"/>
+      <origin xyz="0 0.001 0" rpy="0 0 0"/>
       <geometry>
         <box size="0.030 0.009 0.020"/>
@@ -114,5 +114,5 @@
   <link name="caster_back_left_link">
     <collision>
-      <origin rpy="0 0 0" xyz="0 0 0"/>
+      <origin xyz="0 0.001 0" rpy="0 0 0"/>
       <geometry>
         <box size="0.030 0.009 0.020"/>

Commit message: amended origin of collision in waffle URDF

File: turtlebot3_description/urdf/turtlebot3_waffle.urdf.xacro (robot description, xacro)
@@ -177,5 +177,5 @@
     </visual>
     <collision>
-      <origin xyz="0.003 0.065 0.011" rpy="0 0 0"/>
+      <origin xyz="0.003 0.065 0.007" rpy="0 0 0"/>
       <geometry>
         <box size="0.012 0.132 0.020"/>
