Commit message: change name

File: turtlebot3_description/urdf/turtlebot3_waffle_for_open_manipulator.urdf.xacro (robot description, xacro)
@@ -17,5 +17,5 @@
       <origin xyz="-0.064 0 0.0" rpy="0 0 0"/>
       <geometry>
-        <mesh filename="package://turtlebot3_description/meshes/bases/waffle_base_naked.stl" scale="0.001 0.001 0.001"/>
+        <mesh filename="package://turtlebot3_description/meshes/bases/waffle_base_for_open_manipulator.stl" scale="0.001 0.001 0.001"/>
       </geometry>
       <material name="light_black"/>

File: turtlebot3_description/urdf/turtlebot3_waffle_pi_for_open_manipulator.urdf.xacro (robot description, xacro)
@@ -13,5 +13,5 @@
       <origin xyz="-0.064 0 0.0" rpy="0 0 0"/>
       <geometry>
-        <mesh filename="package://turtlebot3_description/meshes/bases/waffle_pi_base.stl" scale="0.001 0.001 0.001"/>
+        <mesh filename="package://turtlebot3_description/meshes/bases/waffle_pi_base_for_open_manipulator.stl" scale="0.001 0.001 0.001"/>
       </geometry>
       <material name="light_black"/>

Commit message: Updated tb3 for omx urdf files

File: turtlebot3_description/urdf/turtlebot3_waffle_for_open_manipulator.urdf.xacro (robot description, xacro)
@@ -29,8 +29,8 @@
     <inertial>
       <origin xyz="0 0 0" rpy="0 0 0"/>
-      <mass value="1.3729096e+00"/>
-      <inertia ixx="8.7002718e-03" ixy="-4.7576583e-05" ixz="1.1160499e-04"
-               iyy="8.6195418e-03" iyz="-3.5422299e-06"
-               izz="1.4612727e-02" />
+      <mass value="1.6329594e+00"/>
+      <inertia ixx="1.0418769e+05" ixy="1.7327248e+00" ixz="-8.1943898e-01"
+               iyy="1.6997442e+05" iyz="3.9896822e+00"
+               izz="2.2187284e+05" />
     </inertial>
   </link>

File: turtlebot3_description/urdf/turtlebot3_waffle_pi_for_open_manipulator.urdf.xacro (robot description, xacro)
@@ -25,8 +25,8 @@
     <inertial>
       <origin xyz="0 0 0" rpy="0 0 0"/>
-      <mass value="1.3729096e+00"/>
-      <inertia ixx="8.7002718e-03" ixy="-4.7576583e-05" ixz="1.1160499e-04"
-               iyy="8.6195418e-03" iyz="-3.5422299e-06"
-               izz="1.4612727e-02" />
+      <mass value="1.6329594e+00"/>
+      <inertia ixx="1.0418769e+05" ixy="1.7327248e+00" ixz="-8.1943898e-01"
+               iyy="1.6997442e+05" iyz="3.9896822e+00"
+               izz="2.2187284e+05" />
     </inertial>
   </link>

Commit message: updated urdf files

File: turtlebot3_description/urdf/turtlebot3_waffle_for_open_manipulator.urdf.xacro (robot description, xacro)
@@ -2,5 +2,5 @@
 <robot name="turtlebot3_waffle_for_open_manipulator" xmlns:xacro="http://ros.org/wiki/xacro">
   <xacro:include filename="$(find turtlebot3_description)/urdf/common_properties.xacro"/>
-  <xacro:include filename="$(find turtlebot3_description)/urdf/turtlebot3_waffle.gazebo.xacro"/>
+  <xacro:include filename="$(find turtlebot3_description)/urdf/turtlebot3_waffle_pi_for_open_manipulator.gazebo.xacro"/>
   <xacro:property name="r200_cam_rgb_px" value="0.005"/>
   <xacro:property name="r200_cam_rgb_py" value="0.018"/>
@@ -28,9 +28,14 @@
     </collision>
     <inertial>
-      <origin xyz="0 0 0" rpy="0 0 0"/>
-      <mass value="1.6329594e+00"/>
-      <inertia ixx="1.0418769e+05" ixy="1.7327248e+00" ixz="-8.1943898e-01"
-               iyy="1.6997442e+05" iyz="3.9896822e+00"
-               izz="2.2187284e+05" />
+      <!-- <origin xyz="-0.064 0 0" rpy="0 0 0"/> -->
+      <origin xyz="-5.8190646e-02 3.8892103e-02 6.3998774e-02" rpy="0 0 0"/>
+      <mass value="2.7771056e+00"/>
+      <!-- <mass value="1.7771056e+00"/> -->
+      <!-- <inertia ixx="1.8257500e-01" ixy="4.9296089e-03" ixz="-1.1606178e-05" -->
+                <!-- iyy="4.8786869e-02" iyz="1.4954898e-05" -->
+                <!-- izz="3.9852748e-02" /> -->
+      <inertia ixx="1" ixy="0" ixz="0"
+                iyy="1" iyz="0"
+                izz="1" />
     </inertial>
   </link>
