Commit message: add lidar and camera support

File: turtlebot3_description/urdf/turtlebot3_pizza.gazebo.xacro (robot description, xacro)
@@ -86,5 +86,5 @@
       <rightJoint>wheel_right_joint</rightJoint>
       <wheelSeparation>0.46485</wheelSeparation>
-      <wheelDiameter>0.121</wheelDiameter>
+      <wheelDiameter>0.1245</wheelDiameter>
       <wheelAcceleration>1</wheelAcceleration>
       <wheelTorque>10</wheelTorque>
@@ -120,5 +120,5 @@
     </plugin>
   </gazebo>
-  <gazebo reference="base_scan">
+  <!-- <gazebo reference="base_scan">
     <material>Gazebo/FlatBlack</material>
     <sensor type="ray" name="lds_lfcd_sensor">
@@ -151,6 +151,6 @@
       </plugin>
     </sensor>
-  </gazebo>
-  <gazebo reference="camera_rgb_frame">
+  </gazebo> -->
+  <!-- <gazebo reference="camera_rgb_frame">
     <sensor type="depth" name="realsense_R200">
       <always_on>true</always_on>
@@ -194,4 +194,4 @@
       </plugin>
     </sensor>
-  </gazebo>
+  </gazebo> -->
 </robot>

File: turtlebot3_description/urdf/turtlebot3_pizza.urdf.xacro (robot description, xacro)
@@ -5,5 +5,5 @@
   <xacro:include filename="$(find sick_tim)/urdf/sick_tim.urdf.xacro" />
   <xacro:include filename="$(find realsense2_description)/urdf/_d435.urdf.xacro" />
-  <xacro:arg name="use_nominal_extrinsics" default="false"/>
+  <xacro:arg name="use_nominal_extrinsics" default="true"/>
   <xacro:arg name="add_plug" default="false" />
   <xacro:arg name="use_mesh" default="true" />
@@ -23,5 +23,5 @@
       <origin xyz="0.0 0.0 0.0" rpy="0 0 0"/>
       <geometry>
-        <mesh filename="package://turtlebot3_description/meshes/bases/big_base.obj"/>
+        <mesh filename="package://turtlebot3_description/meshes/bases/pizza_base.stl" scale="0.001 0.001 0.001"/>
       </geometry>
       <!-- <material name="light_black"/> -->
@@ -51,12 +51,12 @@
       <origin xyz="0 0 0" rpy="0 0 0"/>
       <geometry>
-        <mesh filename="package://turtlebot3_description/meshes/wheels/big_tire.dae"/>
-      </geometry>
-      <!-- <material name="dark"/> -->
-    </visual>
-    <collision>
-      <origin xyz="0.0 0.0 0" rpy="0 0 0"/>
-      <geometry>
-        <cylinder length="0.02425" radius="0.0605"/>
+        <mesh filename="package://turtlebot3_description/meshes/wheels/pizza_tire.dae"/>
+      </geometry>
+      <!-- <material name="dark"/> -->
+    </visual>
+    <collision>
+      <origin xyz="0.0 0.0 0" rpy="0 0 0"/>
+      <geometry>
+        <cylinder length="0.02425" radius="0.06225"/>
       </geometry>
     </collision>
@@ -79,12 +79,12 @@
       <origin xyz="0 0 0" rpy="0 0 0"/>
       <geometry>
-        <mesh filename="package://turtlebot3_description/meshes/wheels/big_tire.dae"/>
-      </geometry>
-      <!-- <material name="dark"/> -->
-    </visual>
-    <collision>
-      <origin xyz="0.0 0.0 0" rpy="0 0 0"/>
-      <geometry>
-        <cylinder length="0.02425" radius="0.0605"/>
+        <mesh filename="package://turtlebot3_description/meshes/wheels/pizza_tire.dae"/>
+      </geometry>
+      <!-- <material name="dark"/> -->
+    </visual>
+    <collision>
+      <origin xyz="0.0 0.0 0" rpy="0 0 0"/>
+      <geometry>
+        <cylinder length="0.02425" radius="0.06225"/>
       </geometry>
     </collision>
@@ -149,5 +149,5 @@
       <origin xyz="0 0 0" rpy="0 0 0"/>
       <geometry>
-        <mesh filename="package://turtlebot3_description/meshes/joints/big_tire_joint.dae"/>
+        <mesh filename="package://turtlebot3_description/meshes/joints/pizza_tire_joint.dae"/>
       </geometry>
       <!-- <material name="dark"/> -->
@@ -170,5 +170,5 @@
       <origin xyz="0 0 0" rpy="0 0 0"/>
       <geometry>
-        <mesh filename="package://turtlebot3_description/meshes/joints/big_tire_joint.dae"/>
+        <mesh filename="package://turtlebot3_description/meshes/joints/pizza_tire_joint.dae"/>
       </geometry>
       <!-- <material name="dark"/> -->
@@ -191,5 +191,5 @@
       <origin xyz="0 0 0" rpy="0 0 0"/>
       <geometry>
-        <mesh filename="package://turtlebot3_description/meshes/wheels/big_caster.dae"/>
+        <mesh filename="package://turtlebot3_description/meshes/wheels/pizza_caster.dae"/>
       </geometry>
       <!-- <material name="dark"/> -->
@@ -220,5 +220,5 @@
       <origin xyz="0 0 0" rpy="0 0 0"/>
       <geometry>
-        <mesh filename="package://turtlebot3_description/meshes/wheels/big_caster.dae"/>
+        <mesh filename="package://turtlebot3_description/meshes/wheels/pizza_caster.dae"/>
       </geometry>
       <!-- <material name="dark"/> -->
@@ -249,5 +249,5 @@
       <origin xyz="0 0 0" rpy="0 0 0"/>
       <geometry>
-        <mesh filename="package://turtlebot3_description/meshes/joints/big_caster_joint.dae"/>
+        <mesh filename="package://turtlebot3_description/meshes/joints/pizza_caster_joint.dae"/>
       </geometry>
       <!-- <material name="dark"/> -->
@@ -270,5 +270,5 @@
       <origin xyz="0 0 0" rpy="0 0 0"/>
       <geometry>
-        <mesh filename="package://turtlebot3_description/meshes/joints/big_caster_joint.dae"/>
+        <mesh filename="package://turtlebot3_description/meshes/joints/pizza_caster_joint.dae"/>
       </geometry>
       <!-- <material name="dark"/> -->
@@ -287,32 +287,43 @@
   </joint>
   <link name="imu_link"/>
-  <!-- <xacro:sick_tim551 name="laser" ros_topic="scan" > -->
-  <joint name="scan_joint" type="fixed">
-    <parent link="base_link"/>
-    <child link="base_scan"/>
-    <origin xyz="0.09596655 0.0 0.1375" rpy="0 0 ${PI/2}"/>
-  </joint>
-  <link name="base_scan">
-    <visual>
-      <origin xyz="0 0 0" rpy="0 0 0"/>
-      <geometry>
-        <mesh filename="package://turtlebot3_description/meshes/sensors/tim571.stl" scale="0.001 0.001 0.001"/>
-      </geometry>
-      <material name="dark"/>
-    </visual>
-    <collision>
-      <origin xyz="0.015 0 -0.0065" rpy="0 0 0"/>
-      <geometry>
-        <cylinder length="0.0315" radius="0.055"/>
-      </geometry>
-    </collision>
-    <inertial>
-      <mass value="0.114" />
-      <origin xyz="0 0 0" />
-      <inertia ixx="0.001" ixy="0.0" ixz="0.0"
-               iyy="0.001" iyz="0.0"
-               izz="0.001" />
-    </inertial>
-  </link>
+  <joint name="laser_mount_joint" type="fixed">
+    <parent link="base_link"/>
+    <child link="laser_mount_link"/>
+    <origin xyz="0.09496655 0.0 0.1375" rpy="0 0 0"/>
+  </joint>
+  <xacro:sick_tim310 name="laser" ros_topic="scan" />
+  <!-- z_offset: distance between base plate and laser center (= center of mesh) -->
+  <!-- <link name="laser_mount_link">
+    <inertial>
+      <mass value="0.001" />
+      <origin xyz="0 0 0" />
+      <inertia ixx="0.000001" ixy="0.0" ixz="0.0"
+        iyy="0.000001" iyz="0.0" izz="0.000001" />
+    </inertial>
+  </link>
+  <joint name="laser_joint" type="fixed">
+    <parent link="laser_mount_link" />
+    <child link="laser" />
+    <origin rpy="0 0 0" xyz="0 0 0.06296"/>
+  </joint>
+  <link name="laser">
+    <visual>
+      <geometry>
+        <mesh filename="package://sick_tim/meshes/sick_tim551.stl" />
+      </geometry>
+    </visual>
+    <collision>
+      <geometry>
+        <mesh filename="package://sick_tim/meshes/sick_tim551.stl" />
+      </geometry>
+    </collision>
+    there are some problems with inertial parameters of the laser
+    <inertial>
+      <origin xyz="0 0 -0.026" />
+      <inertia ixx="${0.0833333 * 0.250 * (0.06 * 0.06 + 0.086 * 0.086)}" ixy="0.0" ixz="0.0"
+        iyy="${0.0833333 * 0.250 * (0.06 * 0.06 + 0.086 * 0.086)}" iyz="0.0"
+        izz="${0.0833333 * 0.250 * (0.06 * 0.06 + 0.06 * 0.06)}" />
+    </inertial>
+  </link> -->
   <xacro:sensor_d435 parent="base_link" use_nominal_extrinsics="$(arg use_nominal_extrinsics)" add_plug="$(arg add_plug)" use_mesh="$(arg use_mesh)">
     <origin xyz="0.23495003 0.0 0.1490935" rpy="0 0 0"/>

Commit message: fix caster revolution

File: turtlebot3_description/urdf/turtlebot3_pizza.gazebo.xacro (robot description, xacro)
@@ -46,5 +46,5 @@
     <minDepth>0.001</minDepth>
     <maxVel>1.0</maxVel>
-    <!-- <material>Gazebo/FlatBlack</material> -->
+    <material>Gazebo/FlatBlack</material>
   </gazebo>
   <gazebo reference="caster_back_right_link">
@@ -55,7 +55,7 @@
     <minDepth>0.001</minDepth>
     <maxVel>1.0</maxVel>
-    <!-- <material>Gazebo/FlatBlack</material> -->
+    <material>Gazebo/FlatBlack</material>
   </gazebo>
-  <gazebo reference="caster_back_right_conn_link">
+  <gazebo reference="caster_back_left_conn_link">
     <!-- <material>Gazebo/DarkGrey</material> -->
   </gazebo>

File: turtlebot3_description/urdf/turtlebot3_pizza.urdf.xacro (robot description, xacro)
@@ -181,5 +181,5 @@
     </collision> -->
   </link>
-  <joint name="caster_back_left_joint" type="continuous">
+  <joint name="caster_back_left_joint" type="fixed">
     <parent link="base_link"/>
     <child link="caster_back_left_link"/>
@@ -193,5 +193,5 @@
         <mesh filename="package://turtlebot3_description/meshes/wheels/pizza_caster.dae"/>
       </geometry>
-      <!-- <material name="dark"/> -->
+      <material name="dark"/>
     </visual>
     <collision>
@@ -207,8 +207,7 @@
                iyy="0.001" iyz="0.0"
                izz="0.001" />
-      <!-- <inertia ixx="0.000001" ixy="0" ixz="0" iyy="0.000001" iyz="0" izz="0.000001"/> -->
-    </inertial>
-  </link>
-  <joint name="caster_back_right_joint" type="continuous">
+    </inertial>
+  </link>
+  <joint name="caster_back_right_joint" type="fixed">
     <parent link="base_link"/>
     <child link="caster_back_right_link"/>
@@ -222,5 +221,5 @@
         <mesh filename="package://turtlebot3_description/meshes/wheels/pizza_caster.dae"/>
       </geometry>
-      <!-- <material name="dark"/> -->
+      <material name="dark"/>
     </visual>
     <collision>
@@ -236,5 +235,4 @@
                iyy="0.001" iyz="0.0"
                izz="0.001" />
-      <!-- <inertia ixx="0.000001" ixy="0" ixz="0" iyy="0.000001" iyz="0" izz="0.000001"/> -->
     </inertial>
   </link>
