Commit message: delete property

File: turtlebot3_description/urdf/common_properties.xacro (robot description, xacro)
@@ -1,5 +1,4 @@
 <?xml version="1.0" ?>
 <robot name="xacro_properties" xmlns:xacro="http://ros.org/wiki/xacro">
-  <xacro:property name="M_PI" value="3.1415926535897931" />
   <!-- Init colour -->
   <material name="black">

Commit message: add color and camera base

File: turtlebot3_description/urdf/common_properties.xacro (robot description, xacro)
@@ -20,4 +20,7 @@
     <color rgba="0.5 0.5 0.5 1.0"/>
   </material>
+  <material name="light_grey">
+    <color rgba="${211/255} ${211/255} ${211/255} 1.0"/>
+  </material>
   <material name="orange">
     <color rgba="${255/255} ${108/255} ${10/255} 1.0"/>

File: turtlebot3_description/urdf/turtlebot3_pizza.urdf.xacro (robot description, xacro)
@@ -25,5 +25,5 @@
         <mesh filename="package://turtlebot3_description/meshes/bases/pizza_base.stl" scale="0.001 0.001 0.001"/>
       </geometry>
-      <!-- <material name="light_black"/> -->
+      <material name="light_grey"/>
     </visual>
     <collision>
@@ -290,5 +290,5 @@
     <origin xyz="0.09496655 0.0 0.1375" rpy="0 0 0"/>
   </joint>
-  <xacro:sick_tim571 name="laser" ros_topic="scan" />
+  <xacro:sick_tim571 name="laser" ros_topic="scan"/>
   <!-- z_offset: distance between base plate and laser center (= center of mesh) -->
   <!-- <link name="laser_mount_link">
@@ -324,4 +324,18 @@
     </inertial>
   </link> -->
+  <joint name="camera_mount_joint" type="fixed">
+    <parent link="base_link"/>
+    <child link="camera_mount_link"/>
+    <origin xyz="0.210 0.0 0.15148333" rpy="0 0 ${-PI/2}"/>
+  </joint>
+  <link name="camera_mount_link">
+    <visual>
+      <origin xyz="0 0 0" rpy="0 0 0"/>
+      <geometry>
+        <mesh filename="package://turtlebot3_description/meshes/joints/pizza_camera_joint.stl" scale="0.001 0.001 0.001"/>
+      </geometry>
+      <material name="dark"/>
+    </visual>
+  </link>
   <xacro:sensor_d435 parent="base_link" use_nominal_extrinsics="$(arg use_nominal_extrinsics)" add_plug="$(arg add_plug)" use_mesh="$(arg use_mesh)">
     <origin xyz="0.23495003 0.0 0.1490935" rpy="0 0 0"/>
