Commit message: update base_footprint position

File: turtlebot3_description/urdf/turtlebot3_pizza.urdf.xacro (robot description, xacro)
@@ -14,8 +14,22 @@
   <xacro:property name="PI" value="3.14159265358979"/>
   <link name="base_footprint"/>
+  <!-- <joint name="test_joint" type="fixed">
+    <parent link="base_footprint"/>
+    <child link="test_link" />
+    <origin xyz="0.0 0.0 0.0" rpy="0 0 0"/>
+  </joint>
+  <link name="test_link">
+    <visual>
+      <origin xyz="0.0 0.0 0.0" rpy="0 0 0"/>
+      <geometry>
+        <mesh filename="package://turtlebot3_description/meshes/wheels/pizza_tire.dae"/>
+      </geometry>
+      <material name="light_grey"/>
+    </visual>
+  </link> -->
   <joint name="base_joint" type="fixed">
     <parent link="base_footprint"/>
     <child link="base_link" />
-    <origin xyz="0.0 0.0 0.0365" rpy="0 0 0"/>
+    <origin xyz="-0.095 0.0 0.0365" rpy="0 0 0"/>
   </joint>
   <link name="base_link">
@@ -333,11 +347,12 @@
       <origin xyz="0 0 0" rpy="0 0 0"/>
       <geometry>
-        <mesh filename="package://turtlebot3_description/meshes/joints/pizza_camera_joint.stl" scale="0.001 0.001 0.001"/>
+        <mesh filename="package://turtlebot3_description/meshes/joints/pizza_camera_joint.dae"/>
       </geometry>
       <material name="dark"/>
     </visual>
   </link>
-  <xacro:sensor_d435 parent="base_link" use_nominal_extrinsics="$(arg use_nominal_extrinsics)" add_plug="$(arg add_plug)" use_mesh="$(arg use_mesh)">
-    <origin xyz="0.23495003 0.0 0.1490935" rpy="0 0 0"/>
+  <xacro:sensor_d435 parent="camera_mount_link" use_nominal_extrinsics="$(arg use_nominal_extrinsics)" add_plug="$(arg add_plug)" use_mesh="$(arg use_mesh)">
+    <origin xyz="0.0 0.01015 -0.01274993" rpy="0 0 ${PI/2}"/>
+    <!-- <origin xyz="0.23495003 0.0 0.1490935" rpy="0 0 0"/> -->
   </xacro:sensor_d435>
   <!-- <joint name="camera_joint" type="fixed">
