Commit message: update urdf

File: turtlebot3_description/urdf/turtlebot3_big_wheel_for_open_manipulator.urdf.xacro (robot description, xacro)
@@ -3,4 +3,9 @@
   <xacro:include filename="$(find turtlebot3_description)/urdf/common_properties.xacro"/>
   <xacro:include filename="$(find turtlebot3_description)/urdf/turtlebot3_waffle_pi_for_open_manipulator.gazebo.xacro"/>
+  <xacro:arg name="use_nominal_extrinsics" default="true"/>
+  <xacro:arg name="add_plug" default="false" />
+  <xacro:arg name="use_mesh" default="true" />
+  <xacro:arg name="publish_pointcloud" default="false" />
+  <xacro:include filename="$(find realsense2_description)/urdf/_d435.urdf.xacro" />
   <link name="base_footprint"/>
   <joint name="base_joint" type="fixed">
@@ -11,7 +16,7 @@
   <link name="base_link">
     <visual>
-      <origin xyz="-0.064 0 0.0" rpy="0 0 0"/>
-      <geometry>
-        <mesh filename="package://turtlebot3_description/meshes/bases/waffle_pi_base_for_open_manipulator.stl" scale="0.001 0.001 0.001"/>
+      <origin xyz="-0.064 0 0" rpy="0 0 0"/>
+      <geometry>
+        <mesh filename="package://turtlebot3_description/meshes/bases/waffle_pi_base.stl" scale="0.001 0.001 0.001"/>
       </geometry>
       <material name="light_black"/>
@@ -24,12 +29,9 @@
     </collision>
     <inertial>
-      <origin xyz="0.0 0 0.0" rpy="0 0 0"/>
-      <mass value="1.6329594e+00"/>
-      <inertia ixx="1.0" ixy="0.0" ixz="0.0"
-               iyy="1.0" iyz="0.0"
-               izz="1.0" />
-      <!-- <inertia ixx="8.7002718e-03" ixy="-4.7576583e-05" ixz="1.1160499e-04"
+      <origin xyz="0 0 0" rpy="0 0 0"/>
+      <mass value="1.3729096e+00"/>
+      <inertia ixx="8.7002718e-03" ixy="-4.7576583e-05" ixz="1.1160499e-04"
                iyy="8.6195418e-03" iyz="-3.5422299e-06"
-               izz="1.4612727e-02" />                -->
+               izz="1.4612727e-02" />
     </inertial>
   </link>
@@ -77,5 +79,5 @@
     </visual>
     <collision>
-      <origin xyz="0 0.001 0" rpy="0 0 0"/>
+      <origin xyz="0 0 0" rpy="0 0 0"/>
       <geometry>
         <cylinder length="0.02425" radius="0.06225"/>
@@ -93,11 +95,18 @@
     <parent link="base_link"/>
     <child link="caster_back_right_link"/>
-    <origin xyz="-0.177 -0.064 -0.0315" rpy="-1.57 0 0"/>
+    <origin xyz="-0.177 -0.064 0.0" rpy="-1.57 0 0"/>
   </joint>
   <link name="caster_back_right_link">
-    <collision>
-      <origin xyz="0 0.001 0" rpy="0 0 0"/>
-      <geometry>
-        <box size="0.030 0.009 0.020"/>
+    <visual>
+      <origin xyz="0 0.00175 0" rpy="1.57 0 0"/>
+      <geometry>
+        <mesh filename="package://turtlebot3_description/meshes/joints/big_wheel_caster_joint.stl" scale="0.001 0.001 0.001"/>
+      </geometry>
+      <material name="dark"/>
+    </visual>
+    <collision>
+      <origin xyz="0 ${0.039/2} 0" rpy="1.57 0 0"/>
+      <geometry>
+        <box size="0.030 0.009 0.039"/>
       </geometry>
     </collision>
@@ -113,11 +122,18 @@
     <parent link="base_link"/>
     <child link="caster_back_left_link"/>
-    <origin xyz="-0.177 0.064 -0.0315" rpy="-1.57 0 0"/>
+    <origin xyz="-0.177 0.064 0.0" rpy="-1.57 0 0"/>
   </joint>
   <link name="caster_back_left_link">
-    <collision>
-      <origin xyz="0 0.001 0" rpy="0 0 0"/>
-      <geometry>
-        <box size="0.030 0.009 0.020"/>
+    <visual>
+      <origin xyz="0 0.00175 0" rpy="1.57 0 0"/>
+      <geometry>
+        <mesh filename="package://turtlebot3_description/meshes/joints/big_wheel_caster_joint.stl" scale="0.001 0.001 0.001"/>
+      </geometry>
+      <material name="dark"/>
+    </visual>
+    <collision>
+      <origin xyz="0 ${0.039/2} 0" rpy="1.57 0 0"/>
+      <geometry>
+        <box size="0.030 0.009 0.039"/>
       </geometry>
     </collision>
@@ -139,5 +155,5 @@
     <parent link="base_link"/>
     <child link="base_scan"/>
-    <origin xyz="-0.024 0 0.122" rpy="0 0 0"/>
+    <origin xyz="-0.064 0 0.122" rpy="0 0 0"/>
   </joint>
   <link name="base_scan">
@@ -152,5 +168,5 @@
       <origin xyz="0.015 0 -0.0065" rpy="0 0 0"/>
       <geometry>
-        <cylinder length="0.0315" radius="0.045"/>
+        <cylinder length="0.0315" radius="0.055"/>
       </geometry>
     </collision>
@@ -163,5 +179,28 @@
     </inertial>
   </link>
-  <joint name="camera_joint" type="fixed">
+  <joint name="base_camera_joint" type="fixed">
+    <parent link="base_link"/>
+    <child link="base_camera_link"/>
+    <origin xyz="0.039 -0.02958054 0.0915" rpy="0 0 0"/>
+  </joint>
+  <link name="base_camera_link">
+    <visual>
+      <origin xyz="0 0 0.0" rpy="0 0 1.57"/>
+      <geometry>
+        <mesh filename="package://turtlebot3_description/meshes/joints/d435_base_camera.stl" scale="0.001 0.001 0.001"/>
+      </geometry>
+      <material name="light_black"/>
+    </visual>
+    <!-- <collision>
+      <origin xyz="0.015 0 -0.0065" rpy="0 0 0"/>
+      <geometry>
+        <cylinder length="0.0315" radius="0.055"/>
+      </geometry>
+    </collision> -->
+  </link>
+  <xacro:sensor_d435 parent="base_camera_link" use_nominal_extrinsics="$(arg use_nominal_extrinsics)" add_plug="$(arg add_plug)" use_mesh="$(arg use_mesh)">
+    <origin xyz="0.016 0.03 0.0" rpy="0 0 0"/>
+  </xacro:sensor_d435>
+  <!-- <joint name="camera_joint" type="fixed">
     <origin xyz="0.073 -0.011 0.084" rpy="0 0 0"/>
     <parent link="base_link"/>
@@ -187,4 +226,4 @@
     <child link="camera_rgb_optical_frame"/>
   </joint>
-  <link name="camera_rgb_optical_frame"/>
+  <link name="camera_rgb_optical_frame"/> -->
 </robot>

Commit message: update urdf(new pos)

File: turtlebot3_description/urdf/turtlebot3_big_wheel_for_open_manipulator.urdf.xacro (robot description, xacro)
@@ -155,5 +155,5 @@
     <parent link="base_link"/>
     <child link="base_scan"/>
-    <origin xyz="-0.064 0 0.122" rpy="0 0 0"/>
+    <origin xyz="-0.047 0 0.122" rpy="0 0 0"/>
   </joint>
   <link name="base_scan">
@@ -182,5 +182,5 @@
     <parent link="base_link"/>
     <child link="base_camera_link"/>
-    <origin xyz="0.039 -0.02958054 0.0915" rpy="0 0 0"/>
+    <origin xyz="0.045 -0.02958054 0.0915" rpy="0 0 0"/>
   </joint>
   <link name="base_camera_link">

Commit message: update urdf

File: turtlebot3_description/urdf/turtlebot3_big_wheel_for_open_manipulator.urdf.xacro (robot description, xacro)
@@ -2,5 +2,5 @@
 <robot name="turtlebot3_waffle_pi_for_open_manipulator" xmlns:xacro="http://ros.org/wiki/xacro">
   <xacro:include filename="$(find turtlebot3_description)/urdf/common_properties.xacro"/>
-  <xacro:include filename="$(find turtlebot3_description)/urdf/turtlebot3_waffle_pi_for_open_manipulator.gazebo.xacro"/>
+  <xacro:include filename="$(find turtlebot3_description)/urdf/turtlebot3_big_wheel.gazebo.xacro"/>
   <xacro:arg name="use_nominal_extrinsics" default="true"/>
   <xacro:arg name="add_plug" default="false" />
@@ -8,4 +8,5 @@
   <xacro:arg name="publish_pointcloud" default="false" />
   <xacro:include filename="$(find realsense2_description)/urdf/_d435.urdf.xacro" />
+  <xacro:property name="M_PI" value="3.14159265358979"/>
   <link name="base_footprint"/>
   <joint name="base_joint" type="fixed">
@@ -39,5 +40,5 @@
     <parent link="base_link"/>
     <child link="wheel_left_link"/>
-    <origin xyz="0.0 0.144 0.023" rpy="-1.57 0 0"/>
+    <origin xyz="0.0 0.144 0.023" rpy="-${M_PI/2} 0 0"/>
     <axis xyz="0 0 1"/>
   </joint>
@@ -67,5 +68,5 @@
     <parent link="base_link"/>
     <child link="wheel_right_link"/>
-    <origin xyz="0.0 -0.144 0.023" rpy="-1.57 0 0"/>
+    <origin xyz="0.0 -0.144 0.023" rpy="-${M_PI/2} 0 0"/>
     <axis xyz="0 0 1"/>
   </joint>
@@ -95,9 +96,9 @@
     <parent link="base_link"/>
     <child link="caster_back_right_link"/>
-    <origin xyz="-0.177 -0.064 0.0" rpy="-1.57 0 0"/>
+    <origin xyz="-0.177 -0.064 0.0" rpy="-${M_PI/2} 0 0"/>
   </joint>
   <link name="caster_back_right_link">
     <visual>
-      <origin xyz="0 0.00175 0" rpy="1.57 0 0"/>
+      <origin xyz="0 0.00175 0" rpy="${M_PI/2} 0 0"/>
       <geometry>
         <mesh filename="package://turtlebot3_description/meshes/joints/big_wheel_caster_joint.stl" scale="0.001 0.001 0.001"/>
@@ -106,5 +107,5 @@
     </visual>
     <collision>
-      <origin xyz="0 ${0.039/2} 0" rpy="1.57 0 0"/>
+      <origin xyz="0 ${0.039/2} 0" rpy="${M_PI/2} 0 0"/>
       <geometry>
         <box size="0.030 0.009 0.039"/>
@@ -122,9 +123,9 @@
     <parent link="base_link"/>
     <child link="caster_back_left_link"/>
-    <origin xyz="-0.177 0.064 0.0" rpy="-1.57 0 0"/>
+    <origin xyz="-0.177 0.064 0.0" rpy="-${M_PI/2} 0 0"/>
   </joint>
   <link name="caster_back_left_link">
     <visual>
-      <origin xyz="0 0.00175 0" rpy="1.57 0 0"/>
+      <origin xyz="0 0.00175 0" rpy="${M_PI/2} 0 0"/>
       <geometry>
         <mesh filename="package://turtlebot3_description/meshes/joints/big_wheel_caster_joint.stl" scale="0.001 0.001 0.001"/>
@@ -133,5 +134,5 @@
     </visual>
     <collision>
-      <origin xyz="0 ${0.039/2} 0" rpy="1.57 0 0"/>
+      <origin xyz="0 ${0.039/2} 0" rpy="${M_PI/2} 0 0"/>
       <geometry>
         <box size="0.030 0.009 0.039"/>
@@ -182,9 +183,10 @@
     <parent link="base_link"/>
     <child link="base_camera_link"/>
-    <origin xyz="0.045 -0.02958054 0.0915" rpy="0 0 0"/>
+    <origin xyz="0.045 -0.036 0.0915" rpy="0 0 0"/>
+    <!-- <origin xyz="0.045 -0.02958054 0.0915" rpy="0 0 0"/> -->
   </joint>
   <link name="base_camera_link">
     <visual>
-      <origin xyz="0 0 0.0" rpy="0 0 1.57"/>
+      <origin xyz="0 0 0.0" rpy="0 0 ${M_PI/2}"/>
       <geometry>
         <mesh filename="package://turtlebot3_description/meshes/joints/d435_base_camera.stl" scale="0.001 0.001 0.001"/>
@@ -222,5 +224,5 @@
   <link name="camera_rgb_frame"/>
   <joint name="camera_rgb_optical_joint" type="fixed">
-    <origin xyz="0 0 0" rpy="-1.57 0 -1.57"/>
+    <origin xyz="0 0 0" rpy="-${M_PI/2} 0 -${M_PI/2}"/>
     <parent link="camera_rgb_frame"/>
     <child link="camera_rgb_optical_frame"/>
