Commit message: modified the name of bases and model names

File: turtlebot3_description/urdf/turtlebot3_burger.urdf.xacro (robot description, xacro)
@@ -20,5 +20,5 @@
       <origin xyz="0 0 0.0" rpy="0 0 0"/>
       <geometry>
-        <mesh filename="package://turtlebot3_description/meshes/basic_base.stl" scale="0.001 0.001 0.001"/>
+        <mesh filename="package://turtlebot3_description/meshes/bases/burger_base.stl" scale="0.001 0.001 0.001"/>
       </geometry>
       <material name="light_black"/>
@@ -49,5 +49,5 @@
       <origin xyz="0 0 0" rpy="${M_PI*0.5} 0 0"/>
       <geometry>
-        <mesh filename="package://turtlebot3_description/meshes/left_tire.stl" scale="0.001 0.001 0.001"/>
+        <mesh filename="package://turtlebot3_description/meshes/wheels/left_tire.stl" scale="0.001 0.001 0.001"/>
       </geometry>
       <material name="light_black"/>
@@ -77,5 +77,5 @@
       <origin xyz="0 0 0" rpy="${M_PI*0.5} 0 0"/>
       <geometry>
-        <mesh filename="package://turtlebot3_description/meshes/right_tire.stl" scale="0.001 0.001 0.001"/>
+        <mesh filename="package://turtlebot3_description/meshes/wheels/right_tire.stl" scale="0.001 0.001 0.001"/>
       </geometry>
       <material name="light_black"/>

File: turtlebot3_description/urdf/turtlebot3_waffle.urdf.xacro (robot description, xacro)
@@ -27,5 +27,5 @@
       <origin xyz="0 0 0.0" rpy="0 0 0"/>
       <geometry>
-        <mesh filename="package://turtlebot3_description/meshes/premium_base.stl" scale="0.001 0.001 0.001"/>
+        <mesh filename="package://turtlebot3_description/meshes/bases/waffle_base.stl" scale="0.001 0.001 0.001"/>
       </geometry>
       <material name="light_black"/>
@@ -57,5 +57,5 @@
       <origin xyz="0 0 0" rpy="${M_PI*0.5} 0 0"/>
       <geometry>
-        <mesh filename="package://turtlebot3_description/meshes/left_tire.stl" scale="0.001 0.001 0.001"/>
+        <mesh filename="package://turtlebot3_description/meshes/wheels/left_tire.stl" scale="0.001 0.001 0.001"/>
       </geometry>
       <material name="light_black"/>
@@ -85,5 +85,5 @@
       <origin xyz="0 0 0" rpy="${M_PI*0.5} 0 0"/>
       <geometry>
-        <mesh filename="package://turtlebot3_description/meshes/right_tire.stl" scale="0.001 0.001 0.001"/>
+        <mesh filename="package://turtlebot3_description/meshes/wheels/right_tire.stl" scale="0.001 0.001 0.001"/>
       </geometry>
       <material name="light_black"/>

Commit message: modified the materials

File: turtlebot3_description/urdf/turtlebot3_burger.urdf.xacro (robot description, xacro)
@@ -6,6 +6,9 @@
     <color rgba="0.0 0.0 0.0 1.0"/>
   </material>
+  <material name="dark">
+    <color rgba="0.3 0.3 0.3 1.0"/>
+  </material>
   <material name="light_black">
-    <color rgba="0.26 0.28 0.30 1.0"/>
+    <color rgba="0.4 0.4 0.4 1.0"/>
   </material>
   <!-- TurtleBot3 Base-->
@@ -51,5 +54,5 @@
         <mesh filename="package://turtlebot3_description/meshes/wheels/left_tire.stl" scale="0.001 0.001 0.001"/>
       </geometry>
-      <material name="light_black"/>
+      <material name="dark"/>
     </visual>
     <collision>
@@ -79,5 +82,5 @@
         <mesh filename="package://turtlebot3_description/meshes/wheels/right_tire.stl" scale="0.001 0.001 0.001"/>
       </geometry>
-      <material name="light_black"/>
+      <material name="dark"/>
     </visual>
     <collision>
@@ -141,5 +144,5 @@
         <mesh filename="package://turtlebot3_description/meshes/sensors/lds.stl" scale="0.001 0.001 0.001"/>
       </geometry>
-      <material name="light_black"/>
+      <material name="dark"/>
     </visual>
     <collision>

File: turtlebot3_description/urdf/turtlebot3_waffle.urdf.xacro (robot description, xacro)
@@ -13,6 +13,9 @@
     <color rgba="0.0 0.0 0.0 1.0"/>
   </material>
+  <material name="dark">
+    <color rgba="0.3 0.3 0.3 1.0"/>
+  </material>
   <material name="light_black">
-    <color rgba="0.26 0.28 0.30 1.0"/>
+    <color rgba="0.4 0.4 0.4 1.0"/>
   </material>
   <!-- TurtleBot3 Base-->
@@ -59,5 +62,5 @@
         <mesh filename="package://turtlebot3_description/meshes/wheels/left_tire.stl" scale="0.001 0.001 0.001"/>
       </geometry>
-      <material name="light_black"/>
+      <material name="dark"/>
     </visual>
     <collision>
@@ -87,5 +90,5 @@
         <mesh filename="package://turtlebot3_description/meshes/wheels/right_tire.stl" scale="0.001 0.001 0.001"/>
       </geometry>
-      <material name="light_black"/>
+      <material name="dark"/>
     </visual>
     <collision>
@@ -169,5 +172,5 @@
         <mesh filename="package://turtlebot3_description/meshes/sensors/lds.stl" scale="0.001 0.001 0.001"/>
       </geometry>
-      <material name="light_black"/>
+      <material name="dark"/>
     </visual>
     <collision>

Commit message: update urdf and add gazebo

File: turtlebot3_description/urdf/turtlebot3_burger.urdf.xacro (robot description, xacro)
@@ -1,15 +1,6 @@
 <?xml version="1.0" ?>
-<robot name="turtlebot3" xmlns:xacro="http://ros.org/wiki/xacro">
-  <xacro:property name="M_PI" value="3.1415926535897931" />
-  <!-- Init colour -->
-  <material name="black">
-    <color rgba="0.0 0.0 0.0 1.0"/>
-  </material>
-  <material name="dark">
-    <color rgba="0.3 0.3 0.3 1.0"/>
-  </material>
-  <material name="light_black">
-    <color rgba="0.4 0.4 0.4 1.0"/>
-  </material>
+<robot name="turtlebot3_burger" xmlns:xacro="http://ros.org/wiki/xacro">
+  <xacro:include filename="$(find turtlebot3_description)/urdf/common_properties.xacro"/>
+  <xacro:include filename="$(find turtlebot3_description)/urdf/turtlebot3_burger.gazebo"/>
   <!-- TurtleBot3 Base-->
   <link name="base_footprint"/>
@@ -28,7 +19,7 @@
     </visual>
     <collision>
-      <origin xyz="0 0 0" rpy="0 0 0"/>
+      <origin xyz="0 0 0.070" rpy="0 0 0"/>
       <geometry>
-        <box size="0.18 0.12 0.04"/>
+        <box size="0.130 0.130 0.145"/>
       </geometry>
     </collision>
@@ -57,5 +48,5 @@
     </visual>
     <collision>
-      <origin rpy="0 0 0" xyz="0 0 0"/>
+      <origin xyz="0 0 0" rpy="0 0 0"/>
       <geometry>
         <cylinder length="0.018" radius="0.033"/>
@@ -85,5 +76,5 @@
     </visual>
     <collision>
-      <origin rpy="0 0 0" xyz="0 0 0"/>
+      <origin xyz="0 0 0" rpy="0 0 0"/>
       <geometry>
         <cylinder length="0.018" radius="0.033"/>
@@ -98,5 +89,5 @@
     </inertial>
   </link>
-  <joint name="caster_back_joint" type="fixed">
+  <joint name="caster_back_joint" type="continuous">
     <parent link="base_link"/>
     <child link="caster_back_link"/>
@@ -105,7 +96,7 @@
   <link name="caster_back_link">
     <collision>
-      <origin rpy="0 0 0" xyz="0 0 0"/>
+      <origin xyz="0 0 0" rpy="0 0 0"/>
       <geometry>
-        <box size="0.030 0.018 0.010"/>
+        <box size="0.030 0.010 0.020"/>
       </geometry>
     </collision>
@@ -147,7 +138,7 @@
     </visual>
     <collision>
-      <origin rpy="0 0 0" xyz="0 0 0"/>
+      <origin xyz="0 0 0" rpy="0 0 0"/>
       <geometry>
-        <cylinder length="0.0408" radius="0.03785"/>
+        <cylinder length="0.0408" radius="0.050"/>
       </geometry>
     </collision>

File: turtlebot3_description/urdf/turtlebot3_waffle.urdf.xacro (robot description, xacro)
@@ -1,4 +1,6 @@
 <?xml version="1.0" ?>
-<robot name="turtlebot3" xmlns:xacro="http://ros.org/wiki/xacro">
+<robot name="turtlebot3_waffle" xmlns:xacro="http://ros.org/wiki/xacro">
+  <xacro:include filename="$(find turtlebot3_description)/urdf/common_properties.xacro"/>
+  <xacro:include filename="$(find turtlebot3_description)/urdf/turtlebot3_waffle.gazebo"/>
   <xacro:property name="r200_cam_offset_px" value="0.1" />
   <xacro:property name="r200_cam_offset_py" value="-0.028" />
@@ -8,15 +10,4 @@
   <xacro:property name="r200_cam_rgb_pz" value="0.013"/>
   <xacro:property name="r200_cam_depth_offset" value="0.01"/>
-  <xacro:property name="M_PI" value="3.1415926535897931" />
-  <!-- Init colour -->
-  <material name="black">
-    <color rgba="0.0 0.0 0.0 1.0"/>
-  </material>
-  <material name="dark">
-    <color rgba="0.3 0.3 0.3 1.0"/>
-  </material>
-  <material name="light_black">
-    <color rgba="0.4 0.4 0.4 1.0"/>
-  </material>
   <!-- TurtleBot3 Base-->
   <link name="base_footprint"/>
@@ -35,7 +26,7 @@
     </visual>
     <collision>
-      <origin xyz="0 0 0.0" rpy="0 0 0"/>
-      <geometry>
-        <box size="0.266 0.266 0.1"/>
+      <origin xyz="0 0 0.048" rpy="0 0 0"/>
+      <geometry>
+        <box size="0.276 0.256 0.089"/>
       </geometry>
       <material name="light_black"/>
@@ -115,5 +106,5 @@
       <origin rpy="0 0 0" xyz="0 0 0"/>
       <geometry>
-        <box size="0.030 0.018 0.010"/>
+        <box size="0.030 0.010 0.020"/>
       </geometry>
     </collision>
@@ -135,5 +126,5 @@
       <origin rpy="0 0 0" xyz="0 0 0"/>
       <geometry>
-        <box size="0.030 0.018 0.010"/>
+        <box size="0.030 0.010 0.020"/>
       </geometry>
     </collision>
@@ -147,5 +138,5 @@
   </link>
   <!-- TurtleBot3 Sensors-->
-  <joint name="gyro_joint" type="fixed">
+<!--  <joint name="gyro_joint" type="fixed">
     <parent link="base_link"/>
     <child link="gyro_link"/>
@@ -160,5 +151,5 @@
                izz="0.001" />
     </inertial>
-  </link>
+  </link>-->
   <joint name="scan_joint" type="fixed">
     <parent link="base_link"/>
@@ -177,5 +168,5 @@
       <origin rpy="0 0 0" xyz="0 0 0"/>
       <geometry>
-        <cylinder length="0.0408" radius="0.03785"/>
+        <cylinder length="0.0408" radius="0.050"/>
       </geometry>
     </collision>
@@ -201,9 +192,9 @@
     </visual>
     <collision>
-      <origin xyz="0.0 0.0 0.0" rpy="0 0 0"/>
-      <geometry>
-        <box size="0.130 0.567 0.118"/>
-      </geometry>
-    </collision>-->
+      <origin xyz="0.004 0.065 0.009" rpy="0 0 0"/>
+      <geometry>
+        <box size="0.008 0.130 0.019"/>
+      </geometry>
+    </collision>
     <!-- This inertial field needs doesn't contain reliable data!! -->
    <inertial>

Commit message: update stl and urdf

File: turtlebot3_description/urdf/turtlebot3_burger.urdf.xacro (robot description, xacro)
@@ -21,5 +21,5 @@
       <origin xyz="0 0 0.070" rpy="0 0 0"/>
       <geometry>
-        <box size="0.130 0.130 0.145"/>
+        <box size="0.140 0.140 0.145"/>
       </geometry>
     </collision>
@@ -89,5 +89,5 @@
     </inertial>
   </link>
-  <joint name="caster_back_joint" type="continuous">
+  <joint name="caster_back_joint" type="fixed">
     <parent link="base_link"/>
     <child link="caster_back_link"/>
@@ -140,5 +140,5 @@
       <origin xyz="0 0 0" rpy="0 0 0"/>
       <geometry>
-        <cylinder length="0.0408" radius="0.050"/>
+        <cylinder length="0.0408" radius="0.070"/>
       </geometry>
     </collision>

File: turtlebot3_description/urdf/turtlebot3_waffle.urdf.xacro (robot description, xacro)
@@ -28,5 +28,5 @@
       <origin xyz="0 0 0.048" rpy="0 0 0"/>
       <geometry>
-        <box size="0.276 0.256 0.089"/>
+        <box size="0.265 0.265 0.089"/>
       </geometry>
       <material name="light_black"/>
@@ -44,5 +44,5 @@
     <parent link="base_link"/>
     <child link="wheel_left_link"/>
-    <origin xyz="0.064 0.144 0.021" rpy="${-M_PI*0.5} 0 0"/>
+    <origin xyz="0.064 0.144 0.023" rpy="${-M_PI*0.5} 0 0"/>
     <axis xyz="0 0 1"/>
   </joint>
@@ -72,5 +72,5 @@
     <parent link="base_link"/>
     <child link="wheel_right_link"/>
-    <origin xyz="0.064 -0.144 0.021" rpy="${-M_PI*0.5} 0 0"/>
+    <origin xyz="0.064 -0.144 0.023" rpy="${-M_PI*0.5} 0 0"/>
     <axis xyz="0 0 1"/>
   </joint>
@@ -168,5 +168,5 @@
       <origin rpy="0 0 0" xyz="0 0 0"/>
       <geometry>
-        <cylinder length="0.0408" radius="0.050"/>
+        <cylinder length="0.0408" radius="0.070"/>
       </geometry>
     </collision>
@@ -182,5 +182,5 @@
     <origin xyz="0.140 -0.065 0.084" rpy="0 0 0"/>
     <parent link="base_link"/>
-    <child link="camera_link" />
+    <child link="camera_link"/>
   </joint>
   <link name="camera_link">
@@ -192,7 +192,7 @@
     </visual>
     <collision>
-      <origin xyz="0.004 0.065 0.009" rpy="0 0 0"/>
-      <geometry>
-        <box size="0.008 0.130 0.019"/>
+      <origin xyz="0.003 0.065 0.010" rpy="0 0 0"/>
+      <geometry>
+        <box size="0.008 0.130 0.022"/>
       </geometry>
     </collision>
@@ -210,24 +210,24 @@
     <origin xyz="${r200_cam_rgb_px} ${r200_cam_rgb_py} ${r200_cam_rgb_pz}" rpy="0 0 0"/>
     <parent link="camera_link"/>
-    <child link="camera_rgb_frame" />
+    <child link="camera_rgb_frame"/>
   </joint>
   <link name="camera_rgb_frame"/>
   <joint name="camera_rgb_optical_joint" type="fixed">
-    <origin xyz="0 0 0" rpy="${-M_PI/2} 0 ${-M_PI/2}" />
-    <parent link="camera_rgb_frame" />
-    <child link="camera_rgb_optical_frame" />
+    <origin xyz="0 0 0" rpy="${-M_PI/2} 0 ${-M_PI/2}"/>
+    <parent link="camera_rgb_frame"/>
+    <child link="camera_rgb_optical_frame"/>
   </joint>
   <link name="camera_rgb_optical_frame"/>
   <!--Depth joints & links -->
   <joint name="camera_depth_joint" type="fixed">
-      <origin xyz="0 ${r200_cam_depth_offset} 0" rpy="0 0 0" />
-      <parent link="camera_rgb_frame" />
-      <child link="camera_depth_frame" />
+      <origin xyz="0 ${r200_cam_depth_offset} 0" rpy="0 0 0"/>
+      <parent link="camera_rgb_frame"/>
+      <child link="camera_depth_frame"/>
   </joint>
   <link name="camera_depth_frame"/>
   <joint name="camera_depth_optical_joint" type="fixed">
-      <origin xyz="0 0 0" rpy="${-M_PI/2} 0 ${-M_PI/2}" />
-      <parent link="camera_depth_frame" />
-      <child link="camera_depth_optical_frame" />
+      <origin xyz="0 0 0" rpy="${-M_PI/2} 0 ${-M_PI/2}"/>
+      <parent link="camera_depth_frame"/>
+      <child link="camera_depth_optical_frame"/>
   </joint>
   <link name="camera_depth_optical_frame"/>

Commit message: modify footprint

File: turtlebot3_description/urdf/turtlebot3_burger.urdf.xacro (robot description, xacro)
@@ -7,9 +7,9 @@
     <parent link="base_footprint"/>
     <child link="base_link"/>
-    <origin xyz="0 0 0.010" rpy="0 0 0"/>
+    <origin xyz="0.0 0.0 0.010" rpy="0 0 0"/>
   </joint>
   <link name="base_link">
     <visual>
-      <origin xyz="0 0 0.0" rpy="0 0 0"/>
+      <origin xyz="-0.032 0 0.0" rpy="0 0 0"/>
       <geometry>
         <mesh filename="package://turtlebot3_description/meshes/bases/burger_base.stl" scale="0.001 0.001 0.001"/>
@@ -18,7 +18,7 @@
     </visual>
     <collision>
-      <origin xyz="0 0 0.070" rpy="0 0 0"/>
+      <origin xyz="-0.032 0 0.070" rpy="0 0 0"/>
       <geometry>
-        <box size="0.140 0.140 0.145"/>
+        <box size="0.140 0.140 0.140"/>
       </geometry>
     </collision>
@@ -34,5 +34,5 @@
     <parent link="base_link"/>
     <child link="wheel_left_link"/>
-    <origin xyz="0.032 0.08 0.023" rpy="${-M_PI*0.5} 0 0"/>
+    <origin xyz="0.0 0.08 0.023" rpy="${-M_PI*0.5} 0 0"/>
     <axis xyz="0 0 1"/>
   </joint>
@@ -62,5 +62,5 @@
     <parent link="base_link"/>
     <child link="wheel_right_link"/>
-    <origin xyz="0.032 -0.08 0.023" rpy="${-M_PI*0.5} 0 0"/>
+    <origin xyz="0.0 -0.08 0.023" rpy="${-M_PI*0.5} 0 0"/>
     <axis xyz="0 0 1"/>
   </joint>
@@ -90,5 +90,5 @@
     <parent link="base_link"/>
     <child link="caster_back_link"/>
-    <origin xyz="-0.049 0 -0.004" rpy="${-M_PI*0.5} 0 0"/>
+    <origin xyz="-0.081 0 -0.004" rpy="${-M_PI*0.5} 0 0"/>
   </joint>
   <link name="caster_back_link">
@@ -125,5 +125,5 @@
     <parent link="base_link"/>
     <child link="base_scan"/>
-    <origin xyz="0 0 0.171" rpy="0 0 0"/>
+    <origin xyz="-0.032 0 0.171" rpy="0 0 0"/>
   </joint>
   <link name="base_scan">

File: turtlebot3_description/urdf/turtlebot3_waffle.urdf.xacro (robot description, xacro)
@@ -18,5 +18,5 @@
   <link name="base_link">
     <visual>
-      <origin xyz="0 0 0.0" rpy="0 0 0"/>
+      <origin xyz="-0.064 0 0.0" rpy="0 0 0"/>
       <geometry>
         <mesh filename="package://turtlebot3_description/meshes/bases/waffle_base.stl" scale="0.001 0.001 0.001"/>
@@ -25,5 +25,5 @@
     </visual>
     <collision>
-      <origin xyz="0 0 0.048" rpy="0 0 0"/>
+      <origin xyz="-0.064 0 0.048" rpy="0 0 0"/>
       <geometry>
         <box size="0.265 0.265 0.089"/>
@@ -42,5 +42,5 @@
     <parent link="base_link"/>
     <child link="wheel_left_link"/>
-    <origin xyz="0.064 0.144 0.023" rpy="${-M_PI*0.5} 0 0"/>
+    <origin xyz="0.0 0.144 0.023" rpy="${-M_PI*0.5} 0 0"/>
     <axis xyz="0 0 1"/>
   </joint>
@@ -70,5 +70,5 @@
     <parent link="base_link"/>
     <child link="wheel_right_link"/>
-    <origin xyz="0.064 -0.144 0.023" rpy="${-M_PI*0.5} 0 0"/>
+    <origin xyz="0.0 -0.144 0.023" rpy="${-M_PI*0.5} 0 0"/>
     <axis xyz="0 0 1"/>
   </joint>
@@ -98,5 +98,5 @@
     <parent link="base_link"/>
     <child link="caster_back_right_link"/>
-    <origin xyz="-0.113 -0.064 -0.004" rpy="${-M_PI*0.5} 0 0"/>
+    <origin xyz="-0.177 -0.064 -0.004" rpy="${-M_PI*0.5} 0 0"/>
   </joint>
   <link name="caster_back_right_link">
@@ -118,5 +118,5 @@
     <parent link="base_link"/>
     <child link="caster_back_left_link"/>
-    <origin xyz="-0.113 0.064 -0.004" rpy="${-M_PI*0.5} 0 0"/>
+    <origin xyz="-0.177 0.064 -0.004" rpy="${-M_PI*0.5} 0 0"/>
   </joint>
   <link name="caster_back_left_link">
@@ -153,5 +153,5 @@
     <parent link="base_link"/>
     <child link="base_scan"/>
-    <origin xyz="0 0 0.121" rpy="0 0 0"/>
+    <origin xyz="-0.064 0 0.121" rpy="0 0 0"/>
   </joint>
   <link name="base_scan">
@@ -178,5 +178,5 @@
   </link>
   <joint name="camera_joint" type="fixed">
-    <origin xyz="0.140 -0.065 0.084" rpy="0 0 0"/>
+    <origin xyz="0.076 -0.065 0.084" rpy="0 0 0"/>
     <parent link="base_link"/>
     <child link="camera_link"/>
@@ -196,5 +196,5 @@
     </collision>
     <!-- This inertial field needs doesn't contain reliable data!! -->
-   <inertial>
+<!--   <inertial>
       <mass value="0.564" />
       <origin xyz="0 0 0" />
@@ -202,5 +202,5 @@
                iyy="0.000498940" iyz="0.0"
                izz="0.003879257" />
-    </inertial>
+    </inertial>-->
   </link>
   <joint name="camera_rgb_joint" type="fixed">

Commit message: modify inertia

File: turtlebot3_description/urdf/turtlebot3_burger.urdf.xacro (robot description, xacro)
@@ -24,5 +24,5 @@
     </collision>
     <inertial>
-      <origin xyz="0 0 0" rpy="0 0 0"/>
+      <origin xyz="-0.032 0 0" rpy="0 0 0"/>
       <mass value="1"/>
       <inertia ixx="0.01" ixy="0.0" ixz="0.0"

File: turtlebot3_description/urdf/turtlebot3_waffle.urdf.xacro (robot description, xacro)
@@ -32,5 +32,5 @@
     </collision>
     <inertial>
-      <origin xyz="0 0 0" rpy="0 0 0"/>
+      <origin xyz="-0.064 0 0" rpy="0 0 0"/>
       <mass value="1"/>
       <inertia ixx="0.01" ixy="0.0" ixz="0.0"
