Commit message: update height of caster and add mesh

File: turtlebot3_description/urdf/turtlebot3_big_wheel.urdf.xacro (robot description, xacro)
@@ -94,11 +94,18 @@
     <parent link="base_link"/>
     <child link="caster_back_right_link"/>
-    <origin xyz="-0.177 -0.064 -0.0315" rpy="-1.57 0 0"/>
+    <origin xyz="-0.177 -0.064 0.0" rpy="-1.57 0 0"/>
   </joint>
   <link name="caster_back_right_link">
-    <collision>
-      <origin xyz="0 0.001 0" rpy="0 0 0"/>
-      <geometry>
-        <box size="0.030 0.009 0.020"/>
+    <visual>
+      <origin xyz="0 0.00175 0" rpy="1.57 0 0"/>
+      <geometry>
+        <mesh filename="package://turtlebot3_description/meshes/joints/big_wheel_caster_joint.stl" scale="0.001 0.001 0.001"/>
+      </geometry>
+      <material name="dark"/>
+    </visual>
+    <collision>
+      <origin xyz="0 ${0.039/2} 0" rpy="1.57 0 0"/>
+      <geometry>
+        <box size="0.030 0.009 0.039"/>
       </geometry>
     </collision>
@@ -114,11 +121,18 @@
     <parent link="base_link"/>
     <child link="caster_back_left_link"/>
-    <origin xyz="-0.177 0.064 -0.0315" rpy="-1.57 0 0"/>
+    <origin xyz="-0.177 0.064 0.0" rpy="-1.57 0 0"/>
   </joint>
   <link name="caster_back_left_link">
-    <collision>
-      <origin xyz="0 0.001 0" rpy="0 0 0"/>
-      <geometry>
-        <box size="0.030 0.009 0.020"/>
+    <visual>
+      <origin xyz="0 0.00175 0" rpy="1.57 0 0"/>
+      <geometry>
+        <mesh filename="package://turtlebot3_description/meshes/joints/big_wheel_caster_joint.stl" scale="0.001 0.001 0.001"/>
+      </geometry>
+      <material name="dark"/>
+    </visual>
+    <collision>
+      <origin xyz="0 ${0.039/2} 0" rpy="1.57 0 0"/>
+      <geometry>
+        <box size="0.030 0.009 0.039"/>
       </geometry>
     </collision>

Commit message: update urdf

File: turtlebot3_description/urdf/turtlebot3_big_wheel.urdf.xacro (robot description, xacro)
@@ -182,5 +182,5 @@
     <parent link="base_link"/>
     <child link="base_camera_link"/>
-    <origin xyz="0.039 -0.02958054 0.0915" rpy="0 0 0"/>
+    <origin xyz="0.033 -0.02958054 0.0915" rpy="0 0 0"/>
   </joint>
   <link name="base_camera_link">

File: turtlebot3_description/urdf/turtlebot3_big_wheel_3rs.urdf.xacro (robot description, xacro)
@@ -183,5 +183,5 @@
     <parent link="base_link"/>
     <child link="camera_base_front_link"/>
-    <origin xyz="0.033 -0.036 0.0915" rpy="0 0 0"/>
+    <origin xyz="0.039 -0.02958054 0.0915" rpy="0 0 0"/>
   </joint>
   <link name="camera_base_front_link">

File: turtlebot3_description/urdf/turtlebot3_big_wheel_3rs_for_open_manipulator.urdf.xacro (robot description, xacro)
@@ -156,5 +156,5 @@
     <parent link="base_link"/>
     <child link="base_scan"/>
-    <origin xyz="-0.047 0 0.122" rpy="0 0 0"/>
+    <origin xyz="-0.025 0 0.122" rpy="0 0 0"/>
   </joint>
   <link name="base_scan">
@@ -183,5 +183,5 @@
     <parent link="base_link"/>
     <child link="camera_base_front_link"/>
-    <origin xyz="0.045 -0.036 0.0915" rpy="0 0 0"/>
+    <origin xyz="0.039 -0.02958054 0.0915" rpy="0 0 0"/>
     <!-- <origin xyz="0.033 -0.036 0.0915" rpy="0 0 0"/> -->
   </joint>

File: turtlebot3_description/urdf/turtlebot3_big_wheel_for_open_manipulator.urdf.xacro (robot description, xacro)
@@ -156,5 +156,5 @@
     <parent link="base_link"/>
     <child link="base_scan"/>
-    <origin xyz="-0.047 0 0.122" rpy="0 0 0"/>
+    <origin xyz="-0.025 0 0.122" rpy="0 0 0"/>
   </joint>
   <link name="base_scan">
@@ -183,6 +183,6 @@
     <parent link="base_link"/>
     <child link="base_camera_link"/>
-    <origin xyz="0.045 -0.036 0.0915" rpy="0 0 0"/>
-    <!-- <origin xyz="0.045 -0.02958054 0.0915" rpy="0 0 0"/> -->
+    <!-- <origin xyz="0.045 -0.036 0.0915" rpy="0 0 0"/> -->
+    <origin xyz="0.039 -0.02958054 0.0915" rpy="0 0 0"/>
   </joint>
   <link name="base_camera_link">

Commit message: Modified the urdf files for big wheel and big wheel 3rs

File: turtlebot3_description/urdf/turtlebot3_big_wheel.urdf.xacro (robot description, xacro)
@@ -95,5 +95,5 @@
     <parent link="base_link"/>
     <child link="caster_back_right_link"/>
-    <origin xyz="-0.177 -0.064 0.0" rpy="-1.57 0 0"/>
+    <origin xyz="-0.177 -0.064 0.002" rpy="-1.57 0 0"/>
   </joint>
   <link name="caster_back_right_link">
@@ -122,5 +122,5 @@
     <parent link="base_link"/>
     <child link="caster_back_left_link"/>
-    <origin xyz="-0.177 0.064 0.0" rpy="-1.57 0 0"/>
+    <origin xyz="-0.177 0.064 0.002" rpy="-1.57 0 0"/>
   </joint>
   <link name="caster_back_left_link">
@@ -198,4 +198,44 @@
       </geometry>
     </collision> -->
+  </link>
+  <joint name="rpi_joint" type="fixed">
+    <parent link="base_link"/>
+    <child link="rpi_link"/>
+    <origin xyz="-0.13 0.0 0.05" rpy="0 0 0"/>
+  </joint>
+  <link name="rpi_link">
+    <visual>
+      <origin xyz="0 0.00175 0" rpy="0 0 0"/>
+      <geometry>
+        <box size="0.055 0.040 0.02"/>
+      </geometry>
+    </visual>
+    <inertial>
+      <origin xyz="0 0 0"/>
+      <mass value="0.047"/>
+      <inertia ixx="0.001" ixy="0.0" ixz="0.0"
+               iyy="0.001" iyz="0.0"
+               izz="0.001" />
+    </inertial>
+  </link>
+  <joint name="battery_joint" type="fixed">
+    <parent link="base_link"/>
+    <child link="battery_link"/>
+    <origin xyz="-0.13 0.0 0.02" rpy="0 0 0"/>
+  </joint>
+  <link name="battery_link">
+    <visual>
+      <origin xyz="0 0.00175 0" rpy="0 0 0"/>
+      <geometry>
+        <box size="0.08 0.03 0.02"/>
+      </geometry>
+    </visual>
+    <inertial>
+      <origin xyz="0 0 0" />
+      <mass value="0.10" />
+      <inertia ixx="0.001" ixy="0.0" ixz="0.0"
+               iyy="0.001" iyz="0.0"
+               izz="0.001" />
+    </inertial>
   </link>
   <xacro:sensor_d435 parent="base_camera_link" use_nominal_extrinsics="$(arg use_nominal_extrinsics)" add_plug="$(arg add_plug)" use_mesh="$(arg use_mesh)">

File: turtlebot3_description/urdf/turtlebot3_big_wheel_3rs.urdf.xacro (robot description, xacro)
@@ -96,5 +96,5 @@
     <parent link="base_link"/>
     <child link="caster_back_right_link"/>
-    <origin xyz="-0.177 -0.064 0.0" rpy="-${M_PI/2} 0 0"/>
+    <origin xyz="-0.177 -0.064 0.002" rpy="-${M_PI/2} 0 0"/>
   </joint>
   <link name="caster_back_right_link">
@@ -123,5 +123,5 @@
     <parent link="base_link"/>
     <child link="caster_back_left_link"/>
-    <origin xyz="-0.177 0.064 0.0" rpy="-${M_PI/2} 0 0"/>
+    <origin xyz="-0.177 0.064 0.002" rpy="-${M_PI/2} 0 0"/>
   </joint>
   <link name="caster_back_left_link">
@@ -278,4 +278,44 @@
       </geometry>
     </collision> -->
+  </link>
+  <joint name="rpi_joint" type="fixed">
+    <parent link="base_link"/>
+    <child link="rpi_link"/>
+    <origin xyz="-0.13 0.0 0.05" rpy="0 0 0"/>
+  </joint>
+  <link name="rpi_link">
+    <visual>
+      <origin xyz="0 0.00175 0" rpy="0 0 0"/>
+      <geometry>
+        <box size="0.055 0.040 0.02"/>
+      </geometry>
+    </visual>
+    <inertial>
+      <origin xyz="0 0 0"/>
+      <mass value="0.047"/>
+      <inertia ixx="0.001" ixy="0.0" ixz="0.0"
+               iyy="0.001" iyz="0.0"
+               izz="0.001" />
+    </inertial>
+  </link>
+  <joint name="battery_joint" type="fixed">
+    <parent link="base_link"/>
+    <child link="battery_link"/>
+    <origin xyz="-0.13 0.0 0.02" rpy="0 0 0"/>
+  </joint>
+  <link name="battery_link">
+    <visual>
+      <origin xyz="0 0.00175 0" rpy="0 0 0"/>
+      <geometry>
+        <box size="0.08 0.03 0.02"/>
+      </geometry>
+    </visual>
+    <inertial>
+      <origin xyz="0 0 0" />
+      <mass value="0.10" />
+      <inertia ixx="0.001" ixy="0.0" ixz="0.0"
+               iyy="0.001" iyz="0.0"
+               izz="0.001" />
+    </inertial>
   </link>
   <xacro:sensor_d435 parent="camera_base_front_link" name="camera_front" use_nominal_extrinsics="$(arg use_nominal_extrinsics)" add_plug="$(arg add_plug)" use_mesh="$(arg use_mesh)" topics_ns="camera_front">
