Commit message: add 3rs model

File: turtlebot3_description/urdf/turtlebot3_big_wheel_3rs.urdf.xacro (robot description, xacro)
@@ -8,4 +8,5 @@
   <xacro:arg name="publish_pointcloud" default="false" />
   <xacro:include filename="$(find realsense2_description)/urdf/_d435.urdf.xacro" />
+  <xacro:property name="M_PI" value="3.14159265358979"/>
   <link name="base_footprint"/>
   <joint name="base_joint" type="fixed">
@@ -179,14 +180,14 @@
     </inertial>
   </link>
-  <joint name="base_camera_joint" type="fixed">
-    <parent link="base_link"/>
-    <child link="base_camera_link"/>
-    <origin xyz="0.039 -0.02958054 0.0915" rpy="0 0 0"/>
-  </joint>
-  <link name="base_camera_link">
-    <visual>
-      <origin xyz="0 0 0.0" rpy="0 0 1.57"/>
-      <geometry>
-        <mesh filename="package://turtlebot3_description/meshes/joints/d435_base_camera.stl" scale="0.001 0.001 0.001"/>
+  <joint name="camera_base_front_joint" type="fixed">
+    <parent link="base_link"/>
+    <child link="camera_base_front_link"/>
+    <origin xyz="0.033 -0.036 0.0915" rpy="0 0 0"/>
+  </joint>
+  <link name="camera_base_front_link">
+    <visual>
+      <origin xyz="0 0 0" rpy="0 0 ${M_PI/2}"/>
+      <geometry>
+        <mesh filename="package://turtlebot3_description/meshes/joints/d435_camera_base.stl" scale="0.001 0.001 0.001"/>
       </geometry>
       <material name="light_black"/>
@@ -199,6 +200,52 @@
     </collision> -->
   </link>
-  <xacro:sensor_d435 parent="base_camera_link" use_nominal_extrinsics="$(arg use_nominal_extrinsics)" add_plug="$(arg add_plug)" use_mesh="$(arg use_mesh)">
-    <origin xyz="0.016 0.03 0.0" rpy="0 0 0"/>
+  <joint name="camera_base_left_joint" type="fixed">
+    <parent link="base_link"/>
+    <child link="camera_base_left_link"/>
+    <origin xyz="0.028 0.058 0.0915" rpy="0 0 0"/>
+  </joint>
+  <link name="camera_base_left_link">
+    <visual>
+      <origin xyz="0 0 0" rpy="0 0 ${M_PI-0.47560222}"/>
+      <geometry>
+        <mesh filename="package://turtlebot3_description/meshes/joints/d435_camera_base.stl" scale="0.001 0.001 0.001"/>
+      </geometry>
+      <material name="light_black"/>
+    </visual>
+    <!-- <collision>
+      <origin xyz="0.015 0 -0.0065" rpy="0 0 0"/>
+      <geometry>
+        <cylinder length="0.0315" radius="0.055"/>
+      </geometry>
+    </collision> -->
+  </link>
+  <joint name="camera_base_right_joint" type="fixed">
+    <parent link="base_link"/>
+    <child link="camera_base_right_link"/>
+    <origin xyz="-0.036 -0.091 0.0915" rpy="0 0 0"/>
+  </joint>
+  <link name="camera_base_right_link">
+    <visual>
+      <origin xyz="0 0 0" rpy="0 0 0.47560222"/>
+      <geometry>
+        <mesh filename="package://turtlebot3_description/meshes/joints/d435_camera_base.stl" scale="0.001 0.001 0.001"/>
+      </geometry>
+      <material name="light_black"/>
+    </visual>
+    <!-- <collision>
+      <origin xyz="0.015 0 -0.0065" rpy="0 0 0"/>
+      <geometry>
+        <cylinder length="0.0315" radius="0.055"/>
+      </geometry>
+    </collision> -->
+  </link>
+  <xacro:sensor_d435 parent="camera_base_front_link" name="camera_front" use_nominal_extrinsics="$(arg use_nominal_extrinsics)" add_plug="$(arg add_plug)" use_mesh="$(arg use_mesh)" topics_ns="camera_front">
+    <origin xyz="0.016 0.036 0.0" rpy="0 0 0"/>
+  </xacro:sensor_d435>
+  <xacro:sensor_d435 parent="camera_base_left_link" name="camera_left" use_nominal_extrinsics="$(arg use_nominal_extrinsics)" add_plug="$(arg add_plug)" use_mesh="$(arg use_mesh)" topics_ns="camera_left">
+    <origin xyz="-0.02467 0.03070 0.0" rpy="0 0 ${M_PI/2-0.47560222}"/>
+  </xacro:sensor_d435>
+  <xacro:sensor_d435 parent="camera_base_right_link" name="camera_right" use_nominal_extrinsics="$(arg use_nominal_extrinsics)" add_plug="$(arg add_plug)" use_mesh="$(arg use_mesh)" topics_ns="camera_right">
+    <origin xyz="0.03933 0.00225 0.0" rpy="0 0 ${-M_PI/2+0.47560222}"/>
   </xacro:sensor_d435>
   <!-- <joint name="camera_joint" type="fixed">

Commit message: update urdf

File: turtlebot3_description/urdf/turtlebot3_big_wheel_3rs.urdf.xacro (robot description, xacro)
@@ -40,5 +40,5 @@
     <parent link="base_link"/>
     <child link="wheel_left_link"/>
-    <origin xyz="0.0 0.144 0.023" rpy="-1.57 0 0"/>
+    <origin xyz="0.0 0.144 0.023" rpy="-${M_PI/2} 0 0"/>
     <axis xyz="0 0 1"/>
   </joint>
@@ -68,5 +68,5 @@
     <parent link="base_link"/>
     <child link="wheel_right_link"/>
-    <origin xyz="0.0 -0.144 0.023" rpy="-1.57 0 0"/>
+    <origin xyz="0.0 -0.144 0.023" rpy="-${M_PI/2} 0 0"/>
     <axis xyz="0 0 1"/>
   </joint>
@@ -96,9 +96,9 @@
     <parent link="base_link"/>
     <child link="caster_back_right_link"/>
-    <origin xyz="-0.177 -0.064 0.0" rpy="-1.57 0 0"/>
+    <origin xyz="-0.177 -0.064 0.0" rpy="-${M_PI/2} 0 0"/>
   </joint>
   <link name="caster_back_right_link">
     <visual>
-      <origin xyz="0 0.00175 0" rpy="1.57 0 0"/>
+      <origin xyz="0 0.00175 0" rpy="${M_PI/2} 0 0"/>
       <geometry>
         <mesh filename="package://turtlebot3_description/meshes/joints/big_wheel_caster_joint.stl" scale="0.001 0.001 0.001"/>
@@ -107,5 +107,5 @@
     </visual>
     <collision>
-      <origin xyz="0 ${0.039/2} 0" rpy="1.57 0 0"/>
+      <origin xyz="0 ${0.039/2} 0" rpy="${M_PI/2} 0 0"/>
       <geometry>
         <box size="0.030 0.009 0.039"/>
@@ -123,9 +123,9 @@
     <parent link="base_link"/>
     <child link="caster_back_left_link"/>
-    <origin xyz="-0.177 0.064 0.0" rpy="-1.57 0 0"/>
+    <origin xyz="-0.177 0.064 0.0" rpy="-${M_PI/2} 0 0"/>
   </joint>
   <link name="caster_back_left_link">
     <visual>
-      <origin xyz="0 0.00175 0" rpy="1.57 0 0"/>
+      <origin xyz="0 0.00175 0" rpy="${M_PI/2} 0 0"/>
       <geometry>
         <mesh filename="package://turtlebot3_description/meshes/joints/big_wheel_caster_joint.stl" scale="0.001 0.001 0.001"/>
@@ -134,5 +134,5 @@
     </visual>
     <collision>
-      <origin xyz="0 ${0.039/2} 0" rpy="1.57 0 0"/>
+      <origin xyz="0 ${0.039/2} 0" rpy="${M_PI/2} 0 0"/>
       <geometry>
         <box size="0.030 0.009 0.039"/>
@@ -269,5 +269,5 @@
   <link name="camera_rgb_frame"/>
   <joint name="camera_rgb_optical_joint" type="fixed">
-    <origin xyz="0 0 0" rpy="-1.57 0 -1.57"/>
+    <origin xyz="0 0 0" rpy="-${M_PI/2} 0 -${M_PI/2}"/>
     <parent link="camera_rgb_frame"/>
     <child link="camera_rgb_optical_frame"/>

Commit message: update collisions

File: turtlebot3_description/urdf/turtlebot3_big_wheel_3rs.urdf.xacro (robot description, xacro)
@@ -193,4 +193,17 @@
       <material name="light_black"/>
     </visual>
+    <collision>
+      <origin xyz="0 0 0" rpy="0 0 ${M_PI/2}"/>
+      <geometry>
+        <mesh filename="package://turtlebot3_description/meshes/joints/d435_camera_base.stl" scale="0.001 0.001 0.001"/>
+      </geometry>
+    </collision>
+    <inertial>
+      <mass value="0.001" />
+      <origin xyz="0 0 0" />
+      <inertia ixx="0.001" ixy="0.0" ixz="0.0"
+               iyy="0.001" iyz="0.0"
+               izz="0.001" />
+    </inertial>
     <!-- <collision>
       <origin xyz="0.015 0 -0.0065" rpy="0 0 0"/>
@@ -213,4 +226,17 @@
       <material name="light_black"/>
     </visual>
+    <collision>
+      <origin xyz="0 0 0" rpy="0 0 ${M_PI-0.47560222}"/>
+      <geometry>
+        <mesh filename="package://turtlebot3_description/meshes/joints/d435_camera_base.stl" scale="0.001 0.001 0.001"/>
+      </geometry>
+    </collision>
+    <inertial>
+      <mass value="0.001" />
+      <origin xyz="0 0 0" />
+      <inertia ixx="0.001" ixy="0.0" ixz="0.0"
+               iyy="0.001" iyz="0.0"
+               izz="0.001" />
+    </inertial>
     <!-- <collision>
       <origin xyz="0.015 0 -0.0065" rpy="0 0 0"/>
@@ -233,4 +259,17 @@
       <material name="light_black"/>
     </visual>
+    <collision>
+      <origin xyz="0 0 0" rpy="0 0 0.47560222"/>
+      <geometry>
+        <mesh filename="package://turtlebot3_description/meshes/joints/d435_camera_base.stl" scale="0.001 0.001 0.001"/>
+      </geometry>
+    </collision>
+    <inertial>
+      <mass value="0.001" />
+      <origin xyz="0 0 0" />
+      <inertia ixx="0.001" ixy="0.0" ixz="0.0"
+               iyy="0.001" iyz="0.0"
+               izz="0.001" />
+    </inertial>
     <!-- <collision>
       <origin xyz="0.015 0 -0.0065" rpy="0 0 0"/>

File: turtlebot3_description/urdf/turtlebot3_big_wheel_3rs_for_open_manipulator.urdf.xacro (robot description, xacro)
@@ -194,4 +194,17 @@
       <material name="light_black"/>
     </visual>
+    <collision>
+      <origin xyz="0 0 0" rpy="0 0 ${M_PI/2}"/>
+      <geometry>
+        <mesh filename="package://turtlebot3_description/meshes/joints/d435_camera_base.stl" scale="0.001 0.001 0.001"/>
+      </geometry>
+    </collision>
+    <inertial>
+      <mass value="0.001" />
+      <origin xyz="0 0 0" />
+      <inertia ixx="0.001" ixy="0.0" ixz="0.0"
+               iyy="0.001" iyz="0.0"
+               izz="0.001" />
+    </inertial>
     <!-- <collision>
       <origin xyz="0.015 0 -0.0065" rpy="0 0 0"/>
@@ -214,4 +227,17 @@
       <material name="light_black"/>
     </visual>
+    <collision>
+      <origin xyz="0 0 0" rpy="0 0 ${M_PI-0.47560222}"/>
+      <geometry>
+        <mesh filename="package://turtlebot3_description/meshes/joints/d435_camera_base.stl" scale="0.001 0.001 0.001"/>
+      </geometry>
+    </collision>
+    <inertial>
+      <mass value="0.001" />
+      <origin xyz="0 0 0" />
+      <inertia ixx="0.001" ixy="0.0" ixz="0.0"
+               iyy="0.001" iyz="0.0"
+               izz="0.001" />
+    </inertial>
     <!-- <collision>
       <origin xyz="0.015 0 -0.0065" rpy="0 0 0"/>
@@ -234,4 +260,17 @@
       <material name="light_black"/>
     </visual>
+    <collision>
+      <origin xyz="0 0 0" rpy="0 0 0.47560222"/>
+      <geometry>
+        <mesh filename="package://turtlebot3_description/meshes/joints/d435_camera_base.stl" scale="0.001 0.001 0.001"/>
+      </geometry>
+    </collision>
+    <inertial>
+      <mass value="0.001" />
+      <origin xyz="0 0 0" />
+      <inertia ixx="0.001" ixy="0.0" ixz="0.0"
+               iyy="0.001" iyz="0.0"
+               izz="0.001" />
+    </inertial>
     <!-- <collision>
       <origin xyz="0.015 0 -0.0065" rpy="0 0 0"/>

Commit message: Fixed center camera position to be in the center for the URDF file for big wheel 3rs.

File: turtlebot3_description/urdf/turtlebot3_big_wheel_3rs.urdf.xacro (robot description, xacro)
@@ -183,5 +183,5 @@
     <parent link="base_link"/>
     <child link="camera_base_front_link"/>
-    <origin xyz="0.039 -0.02958054 0.0915" rpy="0 0 0"/>
+    <origin xyz="0.033 -0.02958054 0.0915" rpy="0 0 0"/>
   </joint>
   <link name="camera_base_front_link">
@@ -189,5 +189,5 @@
       <origin xyz="0 0 0" rpy="0 0 ${M_PI/2}"/>
       <geometry>
-        <mesh filename="package://turtlebot3_description/meshes/joints/d435_camera_base.stl" scale="0.001 0.001 0.001"/>
+        <mesh filename="package://turtlebot3_description/meshes/joints/d435_base_camera.stl" scale="0.001 0.001 0.001"/>
       </geometry>
       <material name="light_black"/>
@@ -320,5 +320,5 @@
   </link>
   <xacro:sensor_d435 parent="camera_base_front_link" name="camera_front" use_nominal_extrinsics="$(arg use_nominal_extrinsics)" add_plug="$(arg add_plug)" use_mesh="$(arg use_mesh)" topics_ns="camera_front">
-    <origin xyz="0.016 0.036 0.0" rpy="0 0 0"/>
+    <origin xyz="0.016 0.03 0.0" rpy="0 0 0"/>
   </xacro:sensor_d435>
   <xacro:sensor_d435 parent="camera_base_left_link" name="camera_left" use_nominal_extrinsics="$(arg use_nominal_extrinsics)" add_plug="$(arg add_plug)" use_mesh="$(arg use_mesh)" topics_ns="camera_left">

Commit message: Slightly fixed turtlebot3 big wheel 3rs urdf file

File: turtlebot3_description/urdf/turtlebot3_big_wheel_3rs.urdf.xacro (robot description, xacro)
@@ -196,5 +196,5 @@
       <origin xyz="0 0 0" rpy="0 0 ${M_PI/2}"/>
       <geometry>
-        <mesh filename="package://turtlebot3_description/meshes/joints/d435_camera_base.stl" scale="0.001 0.001 0.001"/>
+        <mesh filename="package://turtlebot3_description/meshes/joints/d435_base_camera.stl" scale="0.001 0.001 0.001"/>
       </geometry>
     </collision>
