Commit message: Removed the use of tf_prefix and assigned namespaces to the frame names in the URDF using dynamic variables
Signed-off-by: Hyungyu Kim <kimhg@robotis.com>

File: turtlebot3_description/urdf/turtlebot3_burger.urdf (robot description, URDF)
Before this commit: robot turtlebot3_burger, 7 links, 6 joints
Links:
- removed link base_footprint
- removed link base_link
- removed link base_scan
- removed link caster_back_link
- removed link imu_link
- removed link wheel_left_link
- removed link wheel_right_link
- added link ${namespace}base_footprint
- added link ${namespace}base_link, mass 8.2573504e-01; collision box size=0.140 0.140 0.143; visual mesh filename=package://turtlebot3_description/meshes/bases/burger_base.s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 scale=0.001 0.001 0.001
- added link ${namespace}base_scan, mass 0.114; collision cylinder length=0.0315 radius=0.055; visual mesh filename=package://turtlebot3_description/meshes/sensors/lds.stl scale=0.001 0.001 0.001
- added link ${namespace}caster_back_link, mass 0.005; collision box size=0.030 0.009 0.020
- added link ${namespace}imu_link
- added link ${namespace}wheel_left_link, mass 2.8498940e-02; collision cylinder length=0.018 radius=0.033; visual mesh filename=package://turtlebot3_description/meshes/wheels/left_tire.stl scale=0.001 0.001 0.001
- added link ${namespace}wheel_right_link, mass 2.8498940e-02; collision cylinder length=0.018 radius=0.033; visual mesh filename=package://turtlebot3_description/meshes/wheels/right_tire.s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 scale=0.001 0.001 0.001
Joints:
- removed joint base_joint
- removed joint caster_back_joint
- removed joint imu_joint
- removed joint scan_joint
- removed joint wheel_left_joint
- removed joint wheel_right_joint
- added joint ${namespace}base_joint: type fixed, parent ${namespace}base_footprint, child ${namespace}base_link, origin xyz=0.0 0.0 0.010 rpy=0 0 0
- added joint ${namespace}caster_back_joint: type fixed, parent ${namespace}base_link, child ${namespace}caster_back_link, origin xyz=-0.081 0 -0.004 rpy=-1.57 0 0
- added joint ${namespace}imu_joint: type fixed, parent ${namespace}base_link, child ${namespace}imu_link, origin xyz=-0.032 0 0.068 rpy=0 0 0
- added joint ${namespace}scan_joint: type fixed, parent ${namespace}base_link, child ${namespace}base_scan, origin xyz=-0.032 0 0.172 rpy=0 0 0
- added joint ${namespace}wheel_left_joint: type continuous, parent ${namespace}base_link, child ${namespace}wheel_left_link, origin xyz=0.0 0.08 0.023 rpy=-1.57 0 0, axis 0 0 1
- added joint ${namespace}wheel_right_joint: type continuous, parent ${namespace}base_link, child ${namespace}wheel_right_link, origin xyz=0.0 -0.080 0.023 rpy=-1.57 0 0, axis 0 0 1

File: turtlebot3_description/urdf/turtlebot3_waffle.urdf (robot description, URDF)
Before this commit: robot turtlebot3_waffle, 13 links, 12 joints
Links:
- removed link base_footprint
- removed link base_link
- removed link base_scan
- removed link camera_depth_frame
- removed link camera_depth_optical_frame
- removed link camera_link
- removed link camera_rgb_frame
- removed link camera_rgb_optical_frame
- removed link caster_back_left_link
- removed link caster_back_right_link
- removed link imu_link
- removed link wheel_left_link
- removed link wheel_right_link
- added link ${namespace}base_footprint
- added link ${namespace}base_link, mass 1.3729096e+00; collision box size=0.266 0.266 0.094; visual mesh filename=package://turtlebot3_description/meshes/bases/waffle_base.s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 scale=0.001 0.001 0.001
- added link ${namespace}base_scan, mass 0.114; collision cylinder length=0.0315 radius=0.055; visual mesh filename=package://turtlebot3_description/meshes/sensors/lds.stl scale=0.001 0.001 0.001
- added link ${namespace}camera_depth_frame
- added link ${namespace}camera_depth_optical_frame
- added link ${namespace}camera_link; collision box size=0.012 0.132 0.020; visual mesh filename=package://turtlebot3_description/meshes/sensors/r200.dae
- added link ${namespace}camera_rgb_frame
- added link ${namespace}camera_rgb_optical_frame
- added link ${namespace}caster_back_left_link, mass 0.005; collision box size=0.030 0.009 0.020
- added link ${namespace}caster_back_right_link, mass 0.005; collision box size=0.030 0.009 0.020
- added link ${namespace}imu_link
- added link ${namespace}wheel_left_link, mass 2.8498940e-02; collision cylinder length=0.018 radius=0.033; visual mesh filename=package://turtlebot3_description/meshes/wheels/left_tire.stl scale=0.001 0.001 0.001
- added link ${namespace}wheel_right_link, mass 2.8498940e-02; collision cylinder length=0.018 radius=0.033; visual mesh filename=package://turtlebot3_description/meshes/wheels/right_tire.s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 scale=0.001 0.001 0.001
Joints:
- removed joint base_joint
- removed joint camera_depth_joint
- removed joint camera_depth_optical_joint
- removed joint camera_joint
- removed joint camera_rgb_joint
- removed joint camera_rgb_optical_joint
- removed joint caster_back_left_joint
- removed joint caster_back_right_joint
- removed joint imu_joint
- removed joint scan_joint
- removed joint wheel_left_joint
- removed joint wheel_right_joint
- added joint ${namespace}base_joint: type fixed, parent ${namespace}base_footprint, child ${namespace}base_link, origin xyz=0 0 0.010 rpy=0 0 0
- added joint ${namespace}camera_depth_joint: type fixed, parent ${namespace}camera_link, child ${namespace}camera_depth_frame, origin xyz=0.005 0.028 0.013 rpy=0 0 0
- added joint ${namespace}camera_depth_optical_joint: type fixed, parent ${namespace}camera_depth_frame, child ${namespace}camera_depth_optical_frame, origin xyz=0 0 0 rpy=-1.57 0 -1.57
- added joint ${namespace}camera_joint: type fixed, parent ${namespace}base_link, child ${namespace}camera_link, origin xyz=0.064 -0.065 0.094 rpy=0 0 0
- added joint ${namespace}camera_rgb_joint: type fixed, parent ${namespace}camera_link, child ${namespace}camera_rgb_frame, origin xyz=0.005 0.018 0.013 rpy=0 0 0
- added joint ${namespace}camera_rgb_optical_joint: type fixed, parent ${namespace}camera_rgb_frame, child ${namespace}camera_rgb_optical_frame, origin xyz=0 0 0 rpy=-1.57 0 -1.57
- added joint ${namespace}caster_back_left_joint: type fixed, parent ${namespace}base_link, child ${namespace}caster_back_left_link, origin xyz=-0.177 0.064 -0.004 rpy=-1.57 0 0
- added joint ${namespace}caster_back_right_joint: type fixed, parent ${namespace}base_link, child ${namespace}caster_back_right_link, origin xyz=-0.177 -0.064 -0.004 rpy=-1.57 0 0
- added joint ${namespace}imu_joint: type fixed, parent ${namespace}base_link, child ${namespace}imu_link, origin xyz=0.0 0 0.068 rpy=0 0 0
- added joint ${namespace}scan_joint: type fixed, parent ${namespace}base_link, child ${namespace}base_scan, origin xyz=-0.064 0 0.122 rpy=0 0 0
- added joint ${namespace}wheel_left_joint: type continuous, parent ${namespace}base_link, child ${namespace}wheel_left_link, origin xyz=0.0 0.144 0.023 rpy=-1.57 0 0, axis 0 0 1
- added joint ${namespace}wheel_right_joint: type continuous, parent ${namespace}base_link, child ${namespace}wheel_right_link, origin xyz=0.0 -0.144 0.023 rpy=-1.57 0 0, axis 0 0 1

File: turtlebot3_description/urdf/turtlebot3_waffle_pi.urdf (robot description, URDF)
Before this commit: robot turtlebot3_waffle_pi, 11 links, 10 joints
Links:
- removed link base_footprint
- removed link base_link
- removed link base_scan
- removed link camera_link
- removed link camera_rgb_frame
- removed link camera_rgb_optical_frame
- removed link caster_back_left_link
- removed link caster_back_right_link
- removed link imu_link
- removed link wheel_left_link
- removed link wheel_right_link
- added link ${namespace}base_footprint
- added link ${namespace}base_link, mass 1.3729096e+00; collision box size=0.266 0.266 0.094; visual mesh filename=package://turtlebot3_description/meshes/bases/waffle_pi_bas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 scale=0.001 0.001 0.001
- added link ${namespace}base_scan, mass 0.114; collision cylinder length=0.0315 radius=0.055; visual mesh filename=package://turtlebot3_description/meshes/sensors/lds.stl scale=0.001 0.001 0.001
- added link ${namespace}camera_link; collision box size=0.015 0.030 0.027
- added link ${namespace}camera_rgb_frame
- added link ${namespace}camera_rgb_optical_frame
- added link ${namespace}caster_back_left_link, mass 0.005; collision box size=0.030 0.009 0.020
- added link ${namespace}caster_back_right_link, mass 0.005; collision box size=0.030 0.009 0.020
- added link ${namespace}mu_link
- added link ${namespace}wheel_left_link, mass 2.8498940e-02; collision cylinder length=0.018 radius=0.033; visual mesh filename=package://turtlebot3_description/meshes/wheels/left_tire.stl scale=0.001 0.001 0.001
- added link ${namespace}wheel_right_link, mass 2.8498940e-02; collision cylinder length=0.018 radius=0.033; visual mesh filename=package://turtlebot3_description/meshes/wheels/right_tire.s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 scale=0.001 0.001 0.001
Joints:
- removed joint base_joint
- removed joint camera_joint
- removed joint camera_rgb_joint
- removed joint camera_rgb_optical_joint
- removed joint caster_back_left_joint
- removed joint caster_back_right_joint
- removed joint imu_joint
- removed joint scan_joint
- removed joint wheel_left_joint
- removed joint wheel_right_joint
- added joint ${namespace}base_joint: type fixed, parent ${namespace}base_footprint, child ${namespace}base_link, origin xyz=0 0 0.010 rpy=0 0 0
- added joint ${namespace}camera_joint: type fixed, parent ${namespace}base_link, child ${namespace}camera_link, origin xyz=0.073 -0.011 0.084 rpy=0 0 0
- added joint ${namespace}camera_rgb_joint: type fixed, parent ${namespace}camera_link, child ${namespace}camera_rgb_frame, origin xyz=0.003 0.011 0.009 rpy=0 0 0
- added joint ${namespace}camera_rgb_optical_joint: type fixed, parent ${namespace}camera_rgb_frame, child ${namespace}camera_rgb_optical_frame, origin xyz=0 0 0 rpy=-1.57 0 -1.57
- added joint ${namespace}caster_back_left_joint: type fixed, parent ${namespace}base_link, child ${namespace}caster_back_left_link, origin xyz=-0.177 0.064 -0.004 rpy=-1.57 0 0
- added joint ${namespace}caster_back_right_joint: type fixed, parent ${namespace}base_link, child ${namespace}caster_back_right_link, origin xyz=-0.177 -0.064 -0.004 rpy=-1.57 0 0
- added joint ${namespace}imu_joint: type fixed, parent ${namespace}base_link, child ${namespace}imu_link, origin xyz=0.0 0 0.068 rpy=0 0 0
- added joint ${namespace}scan_joint: type fixed, parent ${namespace}base_link, child ${namespace}base_scan, origin xyz=-0.064 0 0.122 rpy=0 0 0
- added joint ${namespace}wheel_left_joint: type continuous, parent ${namespace}base_link, child ${namespace}wheel_left_link, origin xyz=0.0 0.144 0.023 rpy=-1.57 0 0, axis 0 0 1
- added joint ${namespace}wheel_right_joint: type continuous, parent ${namespace}base_link, child ${namespace}wheel_right_link, origin xyz=0.0 -0.144 0.023 rpy=-1.57 0 0, axis 0 0 1
